File: unnamed/unnamed.kicad_sch (KiCad schematic)
At the start: 128 parts, among them J1 Serial, J2 Serial, J3 Conn_01x01_Female, J4 Conn_01x01_Female, J5 S3B-PH-SM4-TB(LF)(SN), J6 S3B-PH-SM4-TB(LF)(SN), J7 Conn_01x12_Female, J8 Conn_01x12_Female, SW1 SW_Push, SW10 SW_Push, SW11 SW_Push, SW12 SW_Push, SW13 SW_Push, SW14 SW_Push, SW15 SW_Push, SW16 SW_Push, SW17 SW_Push, SW18 SW_Push, SW19 SW_Push, SW2 SW_Push, SW20 SW_Push, SW21 SW_Push, SW22 SW_Push, SW23 SW_Push, SW24 SW_Push, SW25 SW_SPST, SW26 SW_SPST, SW27 SW_Push, SW28 SW_Push, SW29 SW_Push, SW3 SW_Push, SW30 SW_Push, SW31 SW_Push, SW32 SW_Push, SW33 SW_Push, SW34 SW_Push, SW35 SW_Push, SW36 SW_Push, SW4 SW_Push, SW5 SW_Push, SW6 SW_Push, SW7 SW_Push, SW8 SW_Push, SW9 SW_Push, U1 eliteC, U2 eliteC

Commit message: component placement
Parts:
- D10, D13, D14, D15, D18, D19, D20, D24, D25, D26, D3, D30, D33, D4, D5, D8, D9: footprint (none) -> Library:D_1206_handsolder_reversible
Changed lines of the file:
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@@
       (effects (font (size 1.27 1.27)) (justify right))
     )
-    (property "Footprint" "" (id 2) (at 177.8 48.26 0)
+    (property "Footprint" "Library:D_1206_handsolder_reversible" (id 2) (at 177.8 48.26 0)
       (effects (font (size 1.27 1.27)) hide)
     )
@@
       (effects (font (size 1.27 1.27)) (justify right))
     )
-    (property "Footprint" "" (id 2) (at 151.13 58.42 0)
+    (property "Footprint" "Library:D_1206_handsolder_reversible" (id 2) (at 151.13 58.42 0)
       (effects (font (size 1.27 1.27)) hide)
     )
@@
     (property "Reference" "D30" (id 0) (at 217.17 46.99 0))
     (property "Value" "D" (id 1) (at 217.17 49.53 0))
-    (property "Footprint" "" (id 2) (at 217.17 53.34 0)
+    (property "Footprint" "Library:D_1206_handsolder_reversible" (id 2) (at 217.17 53.34 0)
       (effects (font (size 1.27 1.27)) hide)
     )
@@
       (effects (font (size 1.27 1.27)) (justify right))
     )
-    (property "Footprint" "" (id 2) (at 151.13 38.1 0)
+    (property "Footprint" "Library:D_1206_handsolder_reversible" (id 2) (at 151.13 38.1 0)
       (effects (font (size 1.27 1.27)) hide)
     )
@@
       (effects (font (size 1.27 1.27)) (justify right))
     )
-    (property "Footprint" "" (id 2) (at 71.12 58.42 0)
+    (property "Footprint" "Library:D_1206_handsolder_reversible" (id 2) (at 71.12 58.42 0)
       (effects (font (size 1.27 1.27)) hide)
     )
@@
       (effects (font (size 1.27 1.27)) (justify right))
     )
-    (property "Footprint" "" (id 2) (at 124.46 48.26 0)
+    (property "Footprint" "Library:D_1206_handsolder_reversible" (id 2) (at 124.46 48.26 0)
       (effects (font (size 1.27 1.27)) hide)
     )
@@
       (effects (font (size 1.27 1.27)) (justify right))
     )
-    (property "Footprint" "" (id 2) (at 177.8 58.42 0)
+    (property "Footprint" "Library:D_1206_handsolder_reversible" (id 2) (at 177.8 58.42 0)
       (effects (font (size 1.27 1.27)) hide)
     )
@@
       (effects (font (size 1.27 1.27)) (justify right))
     )
-    (property "Footprint" "" (id 2) (at 97.79 48.26 0)
+    (property "Footprint" "Library:D_1206_handsolder_reversible" (id 2) (at 97.79 48.26 0)
       (effects (font (size 1.27 1.27)) hide)
     )
@@
       (effects (font (size 1.27 1.27)) (justify right))
     )
-    (property "Footprint" "" (id 2) (at 97.79 58.42 0)
+    (property "Footprint" "Library:D_1206_handsolder_reversible" (id 2) (at 97.79 58.42 0)
       (effects (font (size 1.27 1.27)) hide)
     )
@@
       (effects (font (size 1.27 1.27)) (justify right))
     )
-    (property "Footprint" "" (id 2) (at 71.12 48.26 0)
+    (property "Footprint" "Library:D_1206_handsolder_reversible" (id 2) (at 71.12 48.26 0)
       (effects (font (size 1.27 1.27)) hide)
     )
@@
       (effects (font (size 1.27 1.27)) (justify right))
     )
-    (property "Footprint" "" (id 2) (at 177.8 38.1 0)
+    (property "Footprint" "Library:D_1206_handsolder_reversible" (id 2) (at 177.8 38.1 0)
       (effects (font (size 1.27 1.27)) hide)
     )
@@
       (effects (font (size 1.27 1.27)) (justify right))
     )
-    (property "Footprint" "" (id 2) (at 124.46 38.1 0)
+    (property "Footprint" "Library:D_1206_handsolder_reversible" (id 2) (at 124.46 38.1 0)
       (effects (font (size 1.27 1.27)) hide)
     )
@@
       (effects (font (size 1.27 1.27)) (justify right))
     )
-    (property "Footprint" "" (id 2) (at 97.79 38.1 0)
+    (property "Footprint" "Library:D_1206_handsolder_reversible" (id 2) (at 97.79 38.1 0)
       (effects (font (size 1.27 1.27)) hide)
     )
@@
       (effects (font (size 1.27 1.27)) (justify right))
     )
-    (property "Footprint" "" (id 2) (at 124.46 58.42 0)
+    (property "Footprint" "Library:D_1206_handsolder_reversible" (id 2) (at 124.46 58.42 0)
       (effects (font (size 1.27 1.27)) hide)
     )
@@
       (effects (font (size 1.27 1.27)) (justify right))
     )
-    (property "Footprint" "" (id 2) (at 71.12 38.1 0)
+    (property "Footprint" "Library:D_1206_handsolder_reversible" (id 2) (at 71.12 38.1 0)
       (effects (font (size 1.27 1.27)) hide)
     )
@@
       (effects (font (size 1.27 1.27)) (justify right))
     )
-    (property "Footprint" "" (id 2) (at 151.13 48.26 0)
+    (property "Footprint" "Library:D_1206_handsolder_reversible" (id 2) (at 151.13 48.26 0)
       (effects (font (size 1.27 1.27)) hide)
     )
@@
     (property "Reference" "D33" (id 0) (at 231.14 46.99 0))
     (property "Value" "D" (id 1) (at 231.14 49.53 0))
-    (property "Footprint" "" (id 2) (at 231.14 53.34 0)
+    (property "Footprint" "Library:D_1206_handsolder_reversible" (id 2) (at 231.14 53.34 0)
       (effects (font (size 1.27 1.27)) hide)
     )
@@
     )
     (path "/bacc65b4-66ed-4f84-a32f-72178fa6b135"
-      (reference "D3") (unit 1) (value "D") (footprint "")
+      (reference "D3") (unit 1) (value "D") (footprint "Library:D_1206_handsolder_reversible")
     )
     (path "/8f8c4061-2489-4125-904b-0f21b5cd5ba1"
-      (reference "D4") (unit 1) (value "D") (footprint "")
+      (reference "D4") (unit 1) (value "D") (footprint "Library:D_1206_handsolder_reversible")
     )
     (path "/53e31bf8-e15b-46dc-88c3-34f753ceba39"
-      (reference "D5") (unit 1) (value "D") (footprint "")
+      (reference "D5") (unit 1) (value "D") (footprint "Library:D_1206_handsolder_reversible")
     )
     (path "/27477966-69c3-4f44-adcc-e25c8b4658ce"
@@
     )
     (path "/acebada4-b199-4d2f-ba15-20b53581e7e9"
-      (reference "D8") (unit 1) (value "D") (footprint "")
+      (reference "D8") (unit 1) (value "D") (footprint "Library:D_1206_handsolder_reversible")
     )
     (path "/6459f10d-9501-43b3-aa58-90a62edefab4"
-      (reference "D9") (unit 1) (value "D") (footprint "")
+      (reference "D9") (unit 1) (value "D") (footprint "Library:D_1206_handsolder_reversible")
     )
     (path "/6a654c93-561f-40fa-b356-527ea5bb0723"
-      (reference "D10") (unit 1) (value "D") (footprint "")
+      (reference "D10") (unit 1) (value "D") (footprint "Library:D_1206_handsolder_reversible")
     )
     (path "/ae1a6041-b452-4a9e-b238-b88c557878b9"
@@
     )
     (path "/9b54bcaf-cfa1-48f1-9831-943fad6af106"
-      (reference "D13") (unit 1) (value "D") (footprint "")
+      (reference "D13") (unit 1) (value "D") (footprint "Library:D_1206_handsolder_reversible")
     )
     (path "/5ea2cc9b-6e4d-47b3-8524-050ee968a948"
-      (reference "D14") (unit 1) (value "D") (footprint "")
+      (reference "D14") (unit 1) (value "D") (footprint "Library:D_1206_handsolder_reversible")
     )
     (path "/b710ca7b-c496-416d-8940-df12f0a94383"
-      (reference "D15") (unit 1) (value "D") (footprint "")
+      (reference "D15") (unit 1) (value "D") (footprint "Library:D_1206_handsolder_reversible")
     )
     (path "/2fb54775-d79c-4284-937b-074a341542c0"
@@
     )
     (path "/48514435-f863-47d9-a8e4-1b0764adb7da"
-      (reference "D18") (unit 1) (value "D") (footprint "")
+      (reference "D18") (unit 1) (value "D") (footprint "Library:D_1206_handsolder_reversible")
     )
     (path "/dd823019-038b-4f3d-b952-8d7ff1ddc521"
-      (reference "D19") (unit 1) (value "D") (footprint "")
+      (reference "D19") (unit 1) (value "D") (footprint "Library:D_1206_handsolder_reversible")
     )
     (path "/0813cd54-c511-4988-96d5-e023e6332984"
-      (reference "D20") (unit 1) (value "D") (footprint "")
+      (reference "D20") (unit 1) (value "D") (footprint "Library:D_1206_handsolder_reversible")
     )
     (path "/98d8f6b8-0b72-4fc1-8947-53e7500e4602"
@@
     )
     (path "/927b8970-34b0-42e3-8893-33c4bb71af0b"
-      (reference "D24") (unit 1) (value "D") (footprint "")
+      (reference "D24") (unit 1) (value "D") (footprint "Library:D_1206_handsolder_reversible")
     )
     (path "/023cb0b1-a0ed-42e7-a84b-f00518aa68e7"
-      (reference "D25") (unit 1) (value "D") (footprint "")
+      (reference "D25") (unit 1) (value "D") (footprint "Library:D_1206_handsolder_reversible")
     )
     (path "/6365e7c9-3d72-4bd0-86b9-c8acb2f4b7f6"
-      (reference "D26") (unit 1) (value "D") (footprint "")
+      (reference "D26") (unit 1) (value "D") (footprint "Library:D_1206_handsolder_reversible")
     )
     (path "/03cb71dc-aa9f-4ef4-9b19-7d6989258e7e"
@@
     )
     (path "/3aa7797a-8b86-4b79-aa68-f8b645c4530e"
-      (reference "D30") (unit 1) (value "D") (footprint "")
+      (reference "D30") (unit 1) (value "D") (footprint "Library:D_1206_handsolder_reversible")
     )
     (path "/3974bbd7-d10d-4b6b-8292-85235e99a6f0"
@@
     )
     (path "/e489aa5e-1344-47ef-aff2-d917d8ea578e"
-      (reference "D33") (unit 1) (value "D") (footprint "")
+      (reference "D33") (unit 1) (value "D") (footprint "Library:D_1206_handsolder_reversible")
     )
     (path "/02b748b1-c67a-406a-a131-8d88b0d498c8"

Commit message: routing
Parts:
- removed J7: Conn_01x12_Female, prettylib:FPC-SMD_FH12-12S-0.5SH-55, symbol Connector:Conn_01x12_Female
- added J7: trackball, Library:6_PinHeader, symbol Connector:Conn_01x06_Female
- added JP1, JP2: Jumper_2_Open, Library:SolderJumper-2_P1.3mm_Open_RoundedPad1.0x1.5mm, symbol Jumper:Jumper_2_Open
- added O3: trackpad, Connector_PinHeader_2.54mm:PinHeader_1x04_P2.54mm_Vertical, symbol Connector_Generic:Conn_01x04
- added R7: 5.1k, Resistor_SMD:R_0402_1005Metric, symbol Device:R
- U2: footprint (none) -> Library:Elite-C
Connections:
- net col1_l is gone; now on net col6_l: U2.18 (F6)
- net row5_l is gone; now on net col3_l: U2.12 (B5)
- net +3V3: now also JP1.2 (B), O3.1 (Pin_1)
- net +5V: now also J7.1 (Pin_1)
- net GND: now also J7.6 (Pin_6), JP2.2 (B)
- net GND2: now also O3.2 (Pin_2)
- net col2_l: now also U2.11 (B4); no longer U2.19 (F5)
- net col3_l: no longer U2.13 (B6)
- net col4_l: now also U2.10 (E6); no longer U2.9 (D7)
- net col5_l: now also U2.9 (D7); no longer U2.10 (E6)
- net col6_l: no longer U2.11 (B4)
- net miso_l: now also J7.5 (Pin_5)
- net mosi_l: now also J7.3 (Pin_3)
- net row1_l: now also U2.19 (F5); no longer U2.20 (F4)
- net row2_l: now also U2.7 (D4); no longer U2.17 (F7)
- net row4_l: now also U2.17 (F7); no longer U2.7 (D4)
- net sc_l: now also J7.4 (Pin_4)
- net scl_l: now also O3.4 (Pin_4)
- net sda_l: now also O3.3 (Pin_3)
- net ss_l: now also U2.13 (B6), J7.2 (Pin_2); no longer U2.29 (F0)
- new net: JP1.1 (A), JP2.1 (A), R7.2
- new net D13: R7.1
- no-connect marks 28 -> 21
Other:
- note added: "Handedness"

Commit message: routing
Parts:
- removed JP1, JP2: Jumper_2_Open, Library:SolderJumper-2_P1.3mm_Open_RoundedPad1.0x1.5mm, symbol Jumper:Jumper_2_Open
- added R8: 5.1k, Resistor_SMD:R_0402_1005Metric, symbol Device:R
Connections:
- net D13 is gone; now on net hand: R7.1
- net +3V3: now also R7.2
- net GND: now also R8.2
- net hand: now reaches U2.20 (F4)
- net hand: now also R8.1
Changed lines of the file:
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@@
   (junction (at 135.89 191.135) (diameter 0) (color 0 0 0 0)
   )
+  (junction (at 296.545 88.9) (diameter 0) (color 0 0 0 0)
+  )
   (junction (at 154.94 206.375) (diameter 0) (color 0 0 0 0)
   )
@@
   (junction (at 55.88 145.415) (diameter 0) (color 0 0 0 0)
   )
-  (junction (at 306.705 88.9) (diameter 0) (color 0 0 0 0)
-  )
   (junction (at 222.25 106.68) (diameter 0) (color 0 0 0 0)
   )
@@
   (no_connect (at 324.485 184.15))
   (no_connect (at 307.975 71.12))
+  (bus_entry (at 81.28 117.475) (size 2.54 2.54)
+    (stroke (width 0) (type default) (color 0 0 0 0))
+  )
   (wire (pts (xy 77.47 198.755) (xy 83.82 198.755))
     (stroke (width 0) (type solid) (color 0 0 0 0))
@@
     (stroke (width 0) (type default) (color 0 0 0 0))
   )
+  (wire (pts (xy 314.96 93.345) (xy 314.96 98.425))
+    (stroke (width 0) (type default) (color 0 0 0 0))
+  )
   (wire (pts (xy 44.45 92.71) (xy 40.64 92.71))
     (stroke (width 0) (type solid) (color 0 0 0 0))
@@
     (stroke (width 0) (type default) (color 0 0 0 0))
   )
-  (wire (pts (xy 304.165 88.9) (xy 306.705 88.9))
+  (wire (pts (xy 304.165 88.9) (xy 318.77 88.9))
     (stroke (width 0) (type default) (color 0 0 0 0))
   )
@@
     (stroke (width 0) (type solid) (color 0 0 0 0))
   )
-  (wire (pts (xy 308.61 98.425) (xy 306.705 98.425))
-    (stroke (width 0) (type default) (color 0 0 0 0))
-  )
   (wire (pts (xy 162.56 99.06) (xy 168.91 99.06))
     (stroke (width 0) (type solid) (color 0 0 0 0))
@@
     (stroke (width 0) (type default) (color 0 0 0 0))
   )
-  (wire (pts (xy 306.705 98.425) (xy 306.705 88.9))
-    (stroke (width 0) (type default) (color 0 0 0 0))
-  )
   (wire (pts (xy 222.25 206.375) (xy 245.11 206.375))
     (stroke (width 0) (type solid) (color 0 0 0 0))
@@
     (stroke (width 0) (type solid) (color 0 0 0 0))
   )
+  (wire (pts (xy 296.545 88.9) (xy 296.545 93.345))
+    (stroke (width 0) (type default) (color 0 0 0 0))
+  )
   (wire (pts (xy 181.61 186.055) (xy 203.2 186.055))
     (stroke (width 0) (type solid) (color 0 0 0 0))
@@
     (stroke (width 0) (type solid) (color 0 0 0 0))
   )
+  (wire (pts (xy 304.165 93.345) (xy 314.96 93.345))
+    (stroke (width 0) (type default) (color 0 0 0 0))
+  )
   (wire (pts (xy 199.39 206.375) (xy 222.25 206.375))
     (stroke (width 0) (type solid) (color 0 0 0 0))
@@
     (stroke (width 0) (type default) (color 0 0 0 0))
   )
-  (wire (pts (xy 306.705 88.9) (xy 308.61 88.9))
-    (stroke (width 0) (type default) (color 0 0 0 0))
-  )
   (wire (pts (xy 135.89 106.68) (xy 154.94 106.68))
     (stroke (width 0) (type default) (color 0 0 0 0))
@@
     (stroke (width 0) (type default) (color 0 0 0 0))
   )
+  (wire (pts (xy 314.96 98.425) (xy 318.77 98.425))
+    (stroke (width 0) (type default) (color 0 0 0 0))
+  )
   (wire (pts (xy 55.88 45.72) (xy 82.55 45.72))
     (stroke (width 0) (type default) (color 0 0 0 0))
@@
     (effects (font (size 1.27 1.27)) (justify left bottom))
   )
-  (label "D13" (at 291.465 88.9 180)
-    (effects (font (size 1.27 1.27)) (justify right bottom))
-  )
   (global_label "row2_r" (shape input) (at 44.45 135.255 180)
     (effects (font (size 1.27 1.27)) (justify right))
@@
     )
   )
+  (global_label "hand" (shape input) (at 318.77 45.72 0) (fields_autoplaced)
+    (effects (font (size 1.27 1.27)) (justify left))
+    (property "Intersheet References" "${INTERSHEET_REFS}" (id 0) (at 325.7793 45.6406 0)
+      (effects (font (size 1.27 1.27)) (justify left) hide)
+    )
+  )
   (global_label "Vcc_r" (shape input) (at 52.07 170.815 180)
     (effects (font (size 1.27 1.27)) (justify right))
@@
     )
   )
+  (global_label "hand" (shape input) (at 291.465 88.9 180) (fields_autoplaced)
+    (effects (font (size 1.27 1.27)) (justify right))
+    (property "Intersheet References" "${INTERSHEET_REFS}" (id 0) (at 284.4557 88.9794 0)
+      (effects (font (size 1.27 1.27)) (justify right) hide)
+    )
+  )
   (global_label "col4_r" (shape input) (at 303.53 168.91 180)
     (effects (font (size 1.27 1.27)) (justify right))
@@
     (pin "4")
   )
-  (symbol (lib_id "Jumper:Jumper_2_Open") (at 313.69 98.425 0) (unit 1)
-    (in_bom yes) (on_board yes) (fields_autoplaced)
-    (property "Reference" "JP2" (id 0) (at 313.69 92.075 0))
-    (property "Value" "Jumper_2_Open" (id 1) (at 313.69 94.615 0))
-    (property "Footprint" "Library:SolderJumper-2_P1.3mm_Open_RoundedPad1.0x1.5mm" (id 2) (at 313.69 98.425 0)
-      (effects (font (size 1.27 1.27)) hide)
-    )
-    (property "Datasheet" "~" (id 3) (at 313.69 98.425 0)
-      (effects (font (size 1.27 1.27)) hide)
-    )
-    (pin "1")
-    (pin "2")
-  )
   (symbol (lib_id "Connector_Generic:Conn_01x04") (at 488.315 40.64 0) (unit 1)
     (in_bom yes) (on_board yes)
@@
     (pin "2")
   )
-  (symbol (lib_id "Jumper:Jumper_2_Open") (at 313.69 88.9 0) (unit 1)
-    (in_bom yes) (on_board yes) (fields_autoplaced)
-    (property "Reference" "JP1" (id 0) (at 313.69 82.55 0))
-    (property "Value" "Jumper_2_Open" (id 1) (at 313.69 85.09 0))
-    (property "Footprint" "Library:SolderJumper-2_P1.3mm_Open_RoundedPad1.0x1.5mm" (id 2) (at 313.69 88.9 0)
-      (effects (font (size 1.27 1.27)) hide)
-    )
-    (property "Datasheet" "~" (id 3) (at 313.69 88.9 0)
-      (effects (font (size 1.27 1.27)) hide)
-    )
-    (pin "1")
-    (pin "2")
-  )
   (symbol (lib_id "Device:D") (at 97.79 38.1 180) (unit 1)
     (in_bom yes) (on_board yes)
@@
     (pin "2")
   )
+  (symbol (lib_id "Device:R") (at 300.355 93.345 90) (unit 1)
+    (in_bom yes) (on_board yes)
+    (property "Reference" "R8" (id 0) (at 299.085 90.805 0)
+      (effects (font (size 1.27 1.27)) (justify left))
+    )
+    (property "Value" "5.1k" (id 1) (at 301.625 90.805 0)
+      (effects (font (size 1.27 1.27)) (justify left))
+    )
+    (property "Footprint" "Resistor_SMD:R_0402_1005Metric" (id 2) (at 300.355 95.123 90)
+      (effects (font (size 1.27 1.27)) hide)
+    )
+    (property "Datasheet" "~" (id 3) (at 300.355 93.345 0)
+      (effects (font (size 1.27 1.27)) hide)
+    )
+    (property "JLCPCB BOM" "1" (id 4) (at 300.355 93.345 0)
+      (effects (font (size 1.27 1.27)) hide)
+    )
+    (property "JLCPCB Part" "C26033" (id 5) (at 300.355 93.345 0)
+      (effects (font (size 1.27 1.27)) hide)
+    )
+    (pin "1")
+    (pin "2")
+  )
   (symbol (lib_id "Device:D") (at 71.12 158.115 180) (unit 1)
     (in_bom yes) (on_board yes)
@@
       (reference "J8") (unit 1) (value "Conn_01x12_Female") (footprint "prettylib:FPC-SMD_FH12-12S-0.5SH-55")
     )
-    (path "/aca14d8b-e103-4ce5-8f9d-018a750e7bdb"
-      (reference "JP1") (unit 1) (value "Jumper_2_Open") (footprint "Library:SolderJumper-2_P1.3mm_Open_RoundedPad1.0x1.5mm")
-    )
-    (path "/799f9801-d8ba-496d-91f3-56c6aceb6340"
-      (reference "JP2") (unit 1) (value "Jumper_2_Open") (footprint "Library:SolderJumper-2_P1.3mm_Open_RoundedPad1.0x1.5mm")
-    )
     (path "/8e810975-a4f5-47c2-90e3-7b00d8f30784"
       (reference "O1") (unit 1) (value "OLED") (footprint "swoop:OLED_jumpers")
@@
       (reference "R7") (unit 1) (value "5.1k") (footprint "Resistor_SMD:R_0402_1005Metric")
     )
+    (path "/fa823f57-7267-4524-bfdd-688b31056389"
+      (reference "R8") (unit 1) (value "5.1k") (footprint "Resistor_SMD:R_0402_1005Metric")
+    )
     (path "/10c00776-633d-4d70-8200-26e4b25fd090"
