File: dilemma/dilemma.kicad_pcb (KiCad board)
At the start: 2 copper layers, 134 x 95.1 mm, 82 parts, among them J1 S3B-PH-SM4-TB(LF)(SN), J2 Serial, J3 BATTERY_CONN_DEANS, J5 S3B-PH-SM4-TB(LF)(SN), SW1 SW_Push, SW10 SW_Push, SW11 SW_Push, SW12 SW_Push, SW13 SW_Push, SW14 SW_Push, SW15 SW_Push, SW16 SW_Push, SW17 locked, SW2 SW_Push, SW26 SW_SPST, SW3 SW_Push, SW37 SW_SPST, SW4 SW_Push, SW5 SW_Push, SW6 SW_Push, SW7 SW_Push, SW8 SW_Push, SW9 SW_Push, U2 eliteC

Commit message: tenting puck
Parts:
- added REF**: Tenting Puck, kbd:Tenting_Puck2, F.Cu at (162.4, 56.6)
- moved D19 5.79 mm to (181.8, 62.1)
- moved D9 4.13 mm to (143.1, 62.1)
- moved D13 0.96 mm to (162.6, 31.9)
- moved D15 0.84 mm to (162.6, 70.6)
Routing:
- net col4_l: track 84.6 -> 80.8 mm
- net Net-(D9-Pad2): track 25.2 -> 28.3 mm
- net col3_l: track 116.3 -> 117.6 mm
- net Net-(D19-Pad2): track 25.5 -> 24.5 mm
- net Net-(D13-Pad2): track 25.2 -> 25.8 mm

Commit message: routing routing routing
Parts:
- removed H3: M4, local-libraries:MountingHole_3mm_Pad_thin
- removed JP9: JUMPER-SMT_3_NO, local-libraries:SolderJumper-3_P1.3mm_Open_RoundedPad1.0x1.5mm_NumberLabels
- added R1: 5.1k, footprints:R_1206_handsolder, F.Cu at (235.5, 43.2)
- R7: footprint local-libraries:R_1206_handsolder_reversible -> footprints:R_1206_handsolder
- moved R7 1.48 mm to (235.5, 43.2), turned to 90 degrees
- turned R3 to -90 degrees
- turned R4 to 90 degrees
Connections:
- J1 pad 1: bat_l -> Gnd_l
- J1 pad 2: Gnd_l -> bat_l
- J5 pad 1: bat_l -> Gnd_l
- J5 pad 2: Gnd_l -> bat_l
- R7 pad 2: Net-(R7-Pad2) -> Vcc_l
- U2 pad 17: row4_l -> row1_l
- U2 pad 19: row1_l -> row4_l
Routing:
- net Gnd_l: track 7.91 -> 138.4 mm, vias 0 -> 4
- net col5_l: track 0.00 -> 123.0 mm
- net serial_l: track 0.00 -> 88.8 mm
- net bat_l: track 7.86 -> 76.3 mm, vias 0 -> 2
- net Vcc_l: track 19.7 -> 87.7 mm, vias 1 -> 3
- net row1_l: track 53.6 -> 119.5 mm
- net sda_l: track 0.00 -> 51.3 mm, vias 0 -> 2
- net scl_l: track 0.00 -> 46.9 mm, vias 1 -> 2
- net col3_l: track 117.6 -> 158.8 mm, vias 1 -> 2
- net col1_l: track 141.3 -> 179.5 mm, vias 1 -> 2
- net Rst_l: track 0.00 -> 35.2 mm, vias 0 -> 1
- net row4_l: track 190.0 -> 219.7 mm
- net row3_l: track 185.4 -> 208.1 mm
- net row2_l: track 173.1 -> 191.3 mm
- net Net-(D33-Pad2): track 24.8 -> 37.8 mm
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
Commit message: silkscreen
Parts:
- removed the kibuzzard-628DFB95 at (271.7, 42.4) (x2)
- added kibuzzard-628DFB95: G***, local-libraries:kibuzzard-628DFB95, F.Cu at (204.9, 96.6)
- added kibuzzard-628DFB95: G***, local-libraries:kibuzzard-628DFB95, B.Cu at (204.9, 96.6)
- moved kibuzzard-61F01A92 64.2 mm to (205.2, 47.7)
- moved G*** 53.1 mm to (221.2, 40.8) (x2)
- moved kibuzzard-61F01A92 10.6 mm to (205.1, 47.8)
- moved kibuzzard-628D3AA1 2.92 mm to (231.6, 43.2)
- moved kibuzzard-61F01C84 2.67 mm to (224.9, 54.2)
- moved JP1 0.17 mm to (216.7, 67.1)
- moved JP2 0.17 mm to (225.3, 67.1)
- moved JP3 0.17 mm to (219.5, 67.1)
- moved JP4 0.17 mm to (222.4, 67.1)
- moved JP5 0.17 mm to (222.4, 67.1)
- moved JP6 0.17 mm to (219.5, 67.1)
- moved JP7 0.17 mm to (225.3, 67.1)
- moved JP8 0.17 mm to (216.7, 67.1)
- moved O2 0.17 mm to (217.2, 71.0)
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Other:
- board text added: "0.1a"

Commit message: drc
Parts:
- removed the kibuzzard-628DFB95 at (204.9, 96.6) (x2)
- added kibuzzard-628DFB95: G***, local-libraries:kibuzzard-628DFB95, F.Cu at (206.2, 96.2)
- added kibuzzard-628DFB95: G***, local-libraries:kibuzzard-628DFB95, B.Cu at (206.2, 96.2)
- moved kibuzzard-61F01C84 2.67 mm to (227.4, 55.2)
- moved kibuzzard-61F01A92 0.46 mm to (205.4, 48.0)
- moved kibuzzard-61F01A92 0.35 mm to (205.6, 47.7)
- moved G*** 0.25 mm to (221.3, 40.6) (x2)
- moved JP1 0.17 mm to (216.7, 67.3)
- moved JP2 0.17 mm to (225.3, 67.3)
- moved JP3 0.17 mm to (219.5, 67.3)
- moved JP4 0.17 mm to (222.4, 67.3)
- moved JP5 0.17 mm to (222.4, 67.3)
- moved JP6 0.17 mm to (219.5, 67.3)
- moved JP7 0.17 mm to (225.3, 67.3)
- moved JP8 0.17 mm to (216.7, 67.3)
- moved O2 0.17 mm to (217.2, 71.2)
- moved kibuzzard-628E0199 0.17 mm to (214.3, 69.5)
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