File: dilemma/0xB2.kicad_pcb (KiCad board)
At the start: 2 copper layers, 134 x 95.1 mm, 127 parts, among them J1 USB_C_Receptacle_USB2.0, J102 Serial, J103 Serial, J104 BATTERY_CONN_DEANS, J105 S3B-PH-SM4-TB(LF)(SN), J106 S3B-PH-SM4-TB(LF)(SN), J5 Conn_01x02, SW1 SW_Push, SW101 SW_Push, SW102 SW_Push, SW103 SW_Push, SW104 SW_Push, SW105 SW_Push, SW106 SW_Push, SW107 SW_Push, SW108 SW_Push, SW109 SW_Push, SW110 SW_SPST, SW111 SW_SPST, SW112 SW_Push, SW113 SW_Push, SW114 SW_Push, SW115 SW_Push, SW116 SW_Push, SW117 SW_Push, SW118 SW_Push, SW119 locked, SW2 SW_Push, U1 RP2040, U101 eliteC, U2 GD25Q80CEIGR, U3 XC6210B332MR-G, Y1 Crystal_GND24

Commit message: routing
Parts:
- removed kibuzzard-628D3AA1: G***, local-libraries:kibuzzard-628D3AA1
- removed rb_cake: G*****, 0xB2_drawings:rb_cake
- removed splinky: G*****, 0xB2_drawings:splinky
- moved kibuzzard-61F01C84 52.0 mm to (149.9, 77.2)
Routing:
- net Gnd_l: track 92.7 -> 30.3 mm, vias 33 -> 28
- net /D15: track 13.9 -> 0.00 mm, vias 1 -> 0
- net /D14: track 11.4 -> 0.00 mm
- net /D12: track 11.3 -> 0.00 mm, vias 1 -> 0
- net /D16: track 10.8 -> 0.00 mm, vias 1 -> 0
- net /D13: track 9.46 -> 0.00 mm
- net sda_l: track 58.0 -> 50.2 mm
- net Vcc_l: track 114.2 -> 118.3 mm, vias 3 -> 4
- net hand: track 11.4 -> 15.2 mm, vias 1 -> 0
- net scl_l: track 49.7 -> 46.6 mm
- net bat_l: track 112.2 -> 111.0 mm
- net Rst_l: track 24.6 -> 23.6 mm
Other:
- board text added: "BastardKB x Freznel x Plut0nium Licensed under CERN-OHL-S v2"
- board text removed: "0xB2"
- board text removed: "BastardKB x Freznel Licensed under CERN-OHL-S v2"
- board text removed: "v3.1"

Commit message: routing, labels
Parts:
- removed U101: eliteC, local-libraries:pro-micro
- removed the kibuzzard-61F01A92 at (77.1, 76.4)
- removed kibuzzard-61F01C84 (x2): G***, local-libraries:kibuzzard-61F01C84
- removed kibuzzard-628D396A: G***, local-libraries:kibuzzard-628D396A
- removed the kibuzzard-628DFB95 at (79.5, 122.8)
- removed kibuzzard-62BF0CBD (x2): G***, kibuzzard-62BF0CBD
- removed kibuzzard-62BF0CFE (x2): G***, kibuzzard-62BF0CFE
- added kibuzzard-62C19A64: G***, kibuzzard-62C19A64, F.Cu at (109.2, 76.8)
- added kibuzzard-62C19A64: G***, kibuzzard-62C19A64, B.Cu at (109.3, 76.8)
- added kibuzzard-62C19AB4: G***, kibuzzard-62C19AB4, F.Cu at (87.4, 97.9)
- added kibuzzard-62C19AC2: G***, kibuzzard-62C19AC2, B.Cu at (87.4, 97.9)
- added kibuzzard-62C19AE7: G***, kibuzzard-62C19AE7, F.Cu at (101.3, 98.3)
- added kibuzzard-62C19AE7: G***, kibuzzard-62C19AE7, B.Cu at (101.3, 98.3)
- kibuzzard-61F01A92: moved to B.Cu
- moved SW110 99.6 mm to (109.2, 71.7)
- moved SW111 99.6 mm to (109.2, 71.7)
- moved kibuzzard-628DFB95 55.2 mm to (94.6, 69.7), turned to 180 degrees
- moved REF** 9.47 mm to (94.7, 79.3)
- moved kibuzzard-61F01A92 6.74 mm to (78.8, 74.6), turned to -90 degrees
- moved R102 4.27 mm to (104.5, 69.8), turned to -90 degrees
- moved R101 4.22 mm to (104.5, 69.7), turned to -90 degrees
- moved JP104 0.11 mm to (98.5, 93.9)
- moved JP105 0.11 mm to (92.8, 93.9)
- moved JP106 0.11 mm to (95.7, 93.9)
- moved JP107 0.11 mm to (95.7, 93.9)
- moved JP108 0.11 mm to (92.8, 93.9)
- moved JP109 0.11 mm to (98.5, 93.9)
- moved O101 0.11 mm to (90.4, 97.8)
- moved JP103 0.11 mm to (89.9, 93.9)
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Routing:
- net bat_l: track 111.0 -> 89.7 mm, vias 4 -> 3
- net mosi_l: track 12.9 -> 0.00 mm, vias 1 -> 0
- net Rst_l: track 23.6 -> 36.3 mm, vias 1 -> 3
- net ss_l: track 12.1 -> 0.00 mm, vias 1 -> 0
- net Vcc_l: track 118.3 -> 128.2 mm, vias 4 -> 5
- net hand: track 15.2 -> 20.4 mm, vias 0 -> 1
- net row4_l: track 231.6 -> 227.7 mm
- net miso_l: track 6.40 -> 2.60 mm
- net row1_l: track 131.9 -> 128.7 mm
- net col5_l: track 133.7 -> 131.0 mm
- net sc_l: track 7.42 -> 5.52 mm
Other:
- board text added: "BastardKB x Freznel x Plut0nium"
- board text removed: "BAT"
- board text removed: "BastardKB x Freznel x Plut0nium Licensed under CERN-OHL-S v2"
- board text removed: "C2"
- board text removed: "C3"
- board text removed: "C4"
- board text removed: "C5"
- board text removed: "C6"
- board text removed: "HAND"
- board text removed: "MISO"
- board text removed: "MOSI"
- board text removed: "R"
- board text removed: "R1"
- board text removed: "R2"
- board text removed: "R3"
- board text removed: "R4"
- board text removed: "RGB"
- board text removed: "RST"
- board text removed: "SC"
- board text removed: "SCL"
- board text removed: "SDA"
- board text removed: "SERIAL"
- board text removed: "SS"
- board text removed: "VCC"

Commit message: FCC
Parts:
- removed the G*** at (13.3, 54.5)
- removed the G*** at (13.4, 54.5)
- D101, D102, D103, D104, D105, D106, D107, D108, D109, D110, D111, D112, D113, D114, D115, D116, D117: footprint local-libraries:D_1206_handsolder_reversible -> local-libraries:R_0402_1005Metric_reversible
- JP107: footprint local-libraries:SolderJumper-2_P1.3mm_Open_RoundedPad1.0x1.5mm -> local-libraries:FPC-SMD_FPC05012-09200-.5mm
- R103: footprint local-libraries:R_1206_handsolder_reversible -> local-libraries:R_0402_1005Metric_nolabel
- R104: footprint local-libraries:R_1206_handsolder_reversible -> local-libraries:R_0402_1005Metric_nolabel; moved to F.Cu
- moved R103 81.9 mm to (151.9, 62.1), turned to 90 degrees
- moved R104 78.1 mm to (150.8, 62.1), turned to -90 degrees
- moved C13 69.1 mm to (164.5, 56.5)
- moved C6 69.1 mm to (162.7, 50.7)
- moved C9 69.1 mm to (153.6, 57.2)
- moved F1 69.1 mm to (156.6, 45.2)
- moved G*** 69.1 mm to (197.3, 23.4) (x2)
- moved J1 69.1 mm to (159.1, 34.2)
- moved J104 69.1 mm to (175.4, 58.3)
- moved J5 69.1 mm to (154.2, 63.8)
- moved PSW101 69.1 mm to (160.6, 83.9)
- moved R10 69.1 mm to (162.7, 49.6)
- moved R101 69.1 mm to (169.2, 45.7)
- moved R2 69.1 mm to (164.1, 60.4)
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Connections:
- net ss_l renamed NCS
Routing:
- net serial_l: track 100.9 -> 61.2 mm, vias 2 -> 0
- net Vcc_l: track 128.2 -> 90.2 mm, vias 5 -> 4
- net scl_l: track 46.6 -> 30.0 mm, vias 2 -> 3
- net sda_l: track 50.2 -> 37.3 mm, vias 2 -> 1
- net Net-(D102-Pad2): track 25.2 -> 27.0 mm
- net col5_l: track 131.0 -> 129.4 mm, vias 1 -> 2
- net col4_l: track 83.0 -> 84.5 mm
- net Net-(D117-Pad2): track 37.8 -> 39.0 mm
- net col2_l: track 125.0 -> 126.2 mm
- net col3_l: track 149.7 -> 148.5 mm
- net Net-(D106-Pad2): track 25.3 -> 26.5 mm
- net col1_l: track 173.4 -> 172.4 mm
- net Net-(D104-Pad2): track 25.4 -> 26.4 mm
- net Net-(D110-Pad2): track 25.7 -> 26.6 mm
- net Net-(D101-Pad2): track 25.2 -> 26.0 mm
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Other:
- outline, holes or cut-outs redrawn
- board text added: "v0.2a"
- board text removed: "0.1b"
- board text removed: "4.7k"
- board text removed: "trackpad pullups"
- board text removed: "v0.1a"

Commit message: ffc
Parts:
- removed R102: 5.1k, footprints:R_1206_handsolder
- added J113: Cirque, local-libraries:FPC-SMD_FPC05012-09200-.5mm, F.Cu at (148.3, 78.7)
- added JP111: Jumper_2_Open, local-libraries:SolderJumper-2_P1.3mm_Open_RoundedPad1.0x1.5mm, B.Cu at (169.0, 69.8)
- added JP112: Jumper_2_Open, local-libraries:SolderJumper-2_P1.3mm_Open_RoundedPad1.0x1.5mm, F.Cu at (169.0, 69.8)
- added kibuzzard-62C1A775: G***, kibuzzard-62C1A775, F.Cu at (169.0, 74.2)
- added kibuzzard-62C1A775: G***, kibuzzard-62C1A775, B.Cu at (169.0, 74.2)
- JP107: footprint local-libraries:FPC-SMD_FPC05012-09200-.5mm -> local-libraries:SolderJumper-2_P1.3mm_Open_RoundedPad1.0x1.5mm
- R101: footprint footprints:R_1206_handsolder -> local-libraries:R_0402_1005Metric_nolabel; moved to F.Cu
- moved JP107 14.7 mm to (160.4, 69.8), turned to -90 degrees
- moved R101 5.67 mm to (167.1, 50.9), turned to 90 degrees
Connections:
- R101 pad 2: Vcc_l -> Net-(R101-Pad2)
Routing:
- net Net-(R101-Pad2): track 0.00 -> 24.0 mm, vias 0 -> 1
- net hand: track 20.4 -> 5.35 mm, vias 1 -> 0
- net scl_l: track 30.0 -> 42.8 mm, vias 3 -> 4
- net sda_l: track 37.3 -> 49.8 mm, vias 1 -> 3
- net Rst_l: track 36.3 -> 33.7 mm
- net bat_l: track 89.7 -> 91.3 mm
- net Vcc_l: track 90.2 -> 91.0 mm, vias 4 -> 3
Other:
- board text removed: "5.1k"
