File: dilemma/0xB2.kicad_pcb (KiCad board)
At the start: 2 copper layers, 134 x 95.1 mm, 122 parts, among them J1 USB_C_Receptacle_USB2.0, J102 Serial, J103 Serial, J104 BATTERY_CONN_DEANS, J105 S3B-PH-SM4-TB(LF)(SN), J106 S3B-PH-SM4-TB(LF)(SN), J113 Cirque, J5 Conn_01x02, SW1 SW_Push, SW101 SW_Push, SW102 SW_Push, SW103 SW_Push, SW104 SW_Push, SW105 SW_Push, SW106 SW_Push, SW107 SW_Push, SW108 SW_Push, SW109 SW_Push, SW110 SW_SPST, SW111 SW_SPST, SW112 SW_Push, SW113 SW_Push, SW114 SW_Push, SW115 SW_Push, SW116 SW_Push, SW117 SW_Push, SW118 SW_Push, SW119 locked, SW2 SW_Push, U1 RP2040, U2 GD25Q80CEIGR, U3 XC6210B332MR-G, Y1 Crystal_GND24

Commit message: silkscreen
Other:
- board text removed: "hands"
Changed lines of the file:
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@@
         (gr_circle (center 0 0.25) (end 0.5 0.25) (width 0) (fill yes))
         (gr_poly (pts
-            (xy 0.5 -0.75)
-            (xy 0 -0.75)
-            (xy 0 0.75)
             (xy 0.5 0.75)
+            (xy 0 0.75)
+            (xy 0 -0.75)
+            (xy 0.5 -0.75)
           ) (width 0) (fill yes))
       ))
@@
         (gr_circle (center 0 0.25) (end 0.5 0.25) (width 0) (fill yes))
         (gr_poly (pts
-            (xy 0 -0.75)
-            (xy -0.5 -0.75)
-            (xy -0.5 0.75)
             (xy 0 0.75)
+            (xy -0.5 0.75)
+            (xy -0.5 -0.75)
+            (xy 0 -0.75)
           ) (width 0) (fill yes))
       ))
@@
     )
     (fp_poly (pts
+        (xy -1.327051 0.029146)
+        (xy -1.184424 0.029146)
+        (xy -1.128691 0.037052)
+        (xy -1.087996 0.060771)
+        (xy -1.054819 0.150068)
+        (xy -1.063346 0.206964)
+        (xy -1.088926 0.251147)
+        (xy -1.129233 0.279673)
+        (xy -1.181943 0.289595)
+        (xy -1.327051 0.289595)
+        (xy -1.327051 0.029146)
+      ) (layer "B.SilkS") (width 0) (fill solid))
+    (fp_poly (pts
         (xy -2.391792 0.775146)
         (xy -1.680518 0.457646)
@@
       ) (layer "B.SilkS") (width 0) (fill solid))
     (fp_poly (pts
-        (xy -1.327051 0.029146)
-        (xy -1.184424 0.029146)
-        (xy -1.128691 0.037052)
-        (xy -1.087996 0.060771)
-        (xy -1.054819 0.150068)
-        (xy -1.063346 0.206964)
-        (xy -1.088926 0.251147)
-        (xy -1.129233 0.279673)
-        (xy -1.181943 0.289595)
-        (xy -1.327051 0.289595)
-        (xy -1.327051 0.029146)
-      ) (layer "B.SilkS") (width 0) (fill solid))
-    (fp_poly (pts
-        (xy 0.36959 -0.108521)
-        (xy 0.563687 -0.108521)
-        (xy 0.466328 0.204639)
-        (xy 0.36959 -0.108521)
-      ) (layer "B.SilkS") (width 0) (fill solid))
-    (fp_poly (pts
         (xy -0.500435 0.289595)
         (xy -0.500435 -0.277813)
@@
         (xy -0.500435 0.289595)
       ) (layer "B.SilkS") (width 0) (fill solid))
+    (fp_poly (pts
+        (xy 0.36959 -0.108521)
+        (xy 0.563687 -0.108521)
+        (xy 0.466328 0.204639)
+        (xy 0.36959 -0.108521)
+      ) (layer "B.SilkS") (width 0) (fill solid))
   )
   (footprint "local-libraries:SolderJumper-2_P1.3mm_Open_RoundedPad1.0x1.5mm" (layer "B.Cu")
@@
     )
     (fp_poly (pts
-        (xy 0.648333 -0.114722)
-        (xy 0.842429 -0.114722)
-        (xy 0.745071 0.198438)
-        (xy 0.648333 -0.114722)
-      ) (layer "B.SilkS") (width 0) (fill solid))
-    (fp_poly (pts
-        (xy -0.612366 0.035347)
-        (xy -0.4747 0.035347)
-        (xy -0.420362 0.043486)
-        (xy -0.381372 0.067903)
-        (xy -0.350056 0.15875)
-        (xy -0.381682 0.250217)
-        (xy -0.42075 0.275099)
-        (xy -0.4747 0.283394)
-        (xy -0.612366 0.283394)
-        (xy -0.612366 0.035347)
-      ) (layer "B.SilkS") (width 0) (fill solid))
-    (fp_poly (pts
         (xy -2.364197 0.781348)
         (xy -2.240406 0.393619)
@@
         (xy -2.364197 0.781348)
       ) (layer "B.SilkS") (width 0) (fill solid))
+    (fp_poly (pts
+        (xy 0.648333 -0.114722)
+        (xy 0.842429 -0.114722)
+        (xy 0.745071 0.198438)
+        (xy 0.648333 -0.114722)
+      ) (layer "B.SilkS") (width 0) (fill solid))
+    (fp_poly (pts
+        (xy -0.612366 0.035347)
+        (xy -0.4747 0.035347)
+        (xy -0.420362 0.043486)
+        (xy -0.381372 0.067903)
+        (xy -0.350056 0.15875)
+        (xy -0.381682 0.250217)
+        (xy -0.42075 0.275099)
+        (xy -0.4747 0.283394)
+        (xy -0.612366 0.283394)
+        (xy -0.612366 0.035347)
+      ) (layer "B.SilkS") (width 0) (fill solid))
   )
   (footprint "local-libraries:Jack_3.5mm_PJ320E_Horizontal_custom" (layer "B.Cu")
@@
   (gr_circle (center 172.52999 38.671819) (end 171.429987 38.671828) (layer "User.7") (width 0.2) (fill none))
   (gr_arc (start 167.520625 64.643485) (mid 168.23994 64.948829) (end 168.520011 65.678356) (layer "User.7") (width 0.2))
-  (gr_text "hands" (at 170.685 46.02 90) (layer "B.SilkS")
-    (effects (font (size 0.8 0.8) (thickness 0.12)) (justify mirror))
-  )
   (gr_text "C3R2" (at 96.775 41.8525) (layer "B.SilkS")
     (effects (font (size 0.8 0.8) (thickness 0.12)) (justify mirror))

Commit message: routing
Routing:
- net mosi_l: track 0.00 -> 42.4 mm, vias 0 -> 2
- net NCS: track 0.00 -> 40.3 mm, vias 0 -> 2
- net miso_l: track 2.60 -> 39.2 mm, vias 0 -> 2
- net sc_l: track 5.52 -> 41.3 mm, vias 0 -> 2
- net Vcc_l: track 91.0 -> 116.6 mm, vias 3 -> 6
- net rgb_l: track 17.8 -> 0.00 mm
- net col2_l: track 126.2 -> 135.5 mm
- net col1_l: track 172.4 -> 180.8 mm
- net col3_l: track 148.5 -> 155.5 mm
- net col4_l: track 84.5 -> 90.9 mm
- net bat_l: track 91.3 -> 87.5 mm
- net row4_l: track 227.7 -> 230.2 mm
- net serial_l: track 61.2 -> 59.2 mm
- net row2_l: track 196.1 -> 197.8 mm
- net sda_l: track 49.8 -> 51.3 mm
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- added copper zone on B.Cu, net Gnd_l
- added copper zone on F.Cu, net Gnd_l
- removed copper zone on B.Cu, net (none)
- removed copper zone on F.Cu, net (none)
- removed copper zone on F.Cu, net Vcc_l

Commit message: drc
Parts:
- moved R4 0.63 mm to (165.0, 43.5), turned to 0 degrees
Connections:
- net Vcc_l renamed +3V3
Routing:
- net Gnd_l: track 30.3 -> 45.0 mm, vias 28 -> 32
- net /LED: track 14.7 -> 11.3 mm
- net sda_l: track 51.3 -> 53.0 mm
- net bat_l: track 87.5 -> 86.2 mm
- added copper zone on F.Cu, net +3V3
