File: dilemma/0xB2.kicad_pcb (KiCad board)
At the start: 2 copper layers, 134 x 95.1 mm, 122 parts, among them J1 USB_C_Receptacle_USB2.0, J102 Serial, J103 Serial, J104 BATTERY_CONN_DEANS, J105 S3B-PH-SM4-TB(LF)(SN), J106 S3B-PH-SM4-TB(LF)(SN), J113 Cirque, J5 Conn_01x02, SW1 SW_Push, SW101 SW_Push, SW102 SW_Push, SW103 SW_Push, SW104 SW_Push, SW105 SW_Push, SW106 SW_Push, SW107 SW_Push, SW108 SW_Push, SW109 SW_Push, SW110 SW_SPST, SW111 SW_SPST, SW112 SW_Push, SW113 SW_Push, SW114 SW_Push, SW115 SW_Push, SW116 SW_Push, SW117 SW_Push, SW118 SW_Push, SW119 locked, SW2 SW_Push, U1 RP2040, U2 GD25Q80CEIGR, U3 XC6210B332MR-G, Y1 Crystal_GND24

Commit message: routing
Routing:
- net Gnd_l: track 55.0 -> 171.8 mm, vias 38 -> 36
- net bat_l: track 86.2 -> 79.0 mm
- net +3V3: track 117.9 -> 120.0 mm
- net col5_l: track 128.8 -> 128.2 mm
- net col1_l: track 180.8 -> 180.3 mm

Commit message: silkscreen
Parts:
- moved kibuzzard-62C19AB4 0.21 mm to (151.9, 73.9)
- moved kibuzzard-62C19AC2 0.19 mm to (151.9, 73.9)
Changed lines of the file:
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@@
       (effects (font (size 1 1) (thickness 0.15)))
     )
-    (fp_line (start 6.4 2.8) (end 1.8 2.8) (layer "B.SilkS") (width 0.12))
-    (fp_line (start 0.3 -9.3) (end 0.3 -12.1) (layer "B.SilkS") (width 0.12))
-    (fp_line (start 0.3 -12.1) (end 6.1 -12.1) (layer "B.SilkS") (width 0.12))
-    (fp_line (start 6.4 -9.3) (end 6.1 -9.3) (layer "B.SilkS") (width 0.12))
-    (fp_line (start 6.1 -9.3) (end 6.1 -12.1) (layer "B.SilkS") (width 0.12))
-    (fp_line (start 6.4 -9.3) (end 6.4 2.8) (layer "B.SilkS") (width 0.12))
-    (fp_line (start -0.9 -9.3) (end -0.9 2.8) (layer "B.SilkS") (width 0.12))
-    (fp_line (start 0.3 -9.3) (end -0.9 -9.3) (layer "B.SilkS") (width 0.12))
-    (fp_line (start -0.9 2.8) (end 1.8 2.8) (layer "B.SilkS") (width 0.12))
-    (fp_line (start -0.9 -9.3) (end -0.9 2.8) (layer "F.SilkS") (width 0.12))
-    (fp_line (start -0.9 2.8) (end 3.7 2.8) (layer "F.SilkS") (width 0.12))
-    (fp_line (start 5.2 -9.3) (end 6.4 -9.3) (layer "F.SilkS") (width 0.12))
-    (fp_line (start 5.2 -12.1) (end -0.6 -12.1) (layer "F.SilkS") (width 0.12))
-    (fp_line (start 6.4 -9.3) (end 6.4 2.8) (layer "F.SilkS") (width 0.12))
-    (fp_line (start -0.9 -9.3) (end -0.6 -9.3) (layer "F.SilkS") (width 0.12))
-    (fp_line (start 6.4 2.8) (end 3.7 2.8) (layer "F.SilkS") (width 0.12))
-    (fp_line (start -0.6 -9.3) (end -0.6 -12.1) (layer "F.SilkS") (width 0.12))
-    (fp_line (start 5.2 -9.3) (end 5.2 -12.1) (layer "F.SilkS") (width 0.12))
-    (fp_line (start 6.8 -12.5) (end 6.8 3) (layer "F.CrtYd") (width 0.05))
-    (fp_line (start -1.3 3) (end 6.8 3) (layer "F.CrtYd") (width 0.05))
     (fp_line (start -1.3 -12.5) (end -1.3 3) (layer "F.CrtYd") (width 0.05))
+    (fp_line (start -1.3 3) (end 6.8 3) (layer "F.CrtYd") (width 0.05))
     (fp_line (start -1.3 -12.5) (end 6.8 -12.5) (layer "F.CrtYd") (width 0.05))
-    (fp_line (start -0.5 -9.2) (end -0.5 -12) (layer "F.Fab") (width 0.1))
+    (fp_line (start 6.8 -12.5) (end 6.8 3) (layer "F.CrtYd") (width 0.05))
     (fp_line (start -0.8 -9.2) (end -0.5 -9.2) (layer "F.Fab") (width 0.1))
-    (fp_line (start 5.1 -9.2) (end 6.3 -9.2) (layer "F.Fab") (width 0.1))
-    (fp_line (start -0.5 -12) (end 5.1 -12) (layer "F.Fab") (width 0.1))
     (fp_line (start 3.7 2) (end -0.8 2) (layer "F.Fab") (width 0.1))
+    (fp_line (start 5.1 -9.2) (end 6.3 -9.2) (layer "F.Fab") (width 0.1))
     (fp_line (start 5.1 -12) (end 5.1 -9.2) (layer "F.Fab") (width 0.1))
-    (fp_line (start -0.8 2) (end -0.8 -9.2) (layer "F.Fab") (width 0.1))
-    (fp_line (start 6.3 -9.2) (end 6.3 2) (layer "F.Fab") (width 0.1))
     (fp_line (start 6.3 2) (end 5.3 2) (layer "F.Fab") (width 0.1))
+    (fp_line (start 6.3 -9.2) (end 6.3 2) (layer "F.Fab") (width 0.1))
+    (fp_line (start -0.5 -12) (end 5.1 -12) (layer "F.Fab") (width 0.1))
+    (fp_line (start -0.8 2) (end -0.8 -9.2) (layer "F.Fab") (width 0.1))
+    (fp_line (start -0.5 -9.2) (end -0.5 -12) (layer "F.Fab") (width 0.1))
     (fp_circle (center 0.9 0) (end 1.2 0.15) (layer "F.Fab") (width 0.12) (fill none))
     (pad "" np_thru_hole oval (at 2.3 -1.6 180) (size 1.5 1.5) (drill oval 1.5) (layers *.Cu *.Mask))
@@
       (effects (font (size 1 1) (thickness 0.15)))
     )
-    (fp_line (start 1.33 -1.237931) (end 1.33 8.95) (layer "B.SilkS") (width 0.12))
-    (fp_line (start -1.33 -1.237931) (end -1.33 8.95) (layer "B.SilkS") (width 0.12))
-    (fp_line (start 1.33 -1.237931) (end -1.33 -1.237931) (layer "B.SilkS") (width 0.12))
-    (fp_line (start 1.33 8.95) (end -1.33 8.95) (layer "B.SilkS") (width 0.12))
-    (fp_line (start -1.33 8.95) (end 1.33 8.95) (layer "F.SilkS") (width 0.12))
-    (fp_line (start -1.33 -1.237931) (end 1.33 -1.237931) (layer "F.SilkS") (width 0.12))
-    (fp_line (start -1.33 -1.237931) (end -1.33 8.95) (layer "F.SilkS") (width 0.12))
-    (fp_line (start 1.33 -1.237931) (end 1.33 8.95) (layer "F.SilkS") (width 0.12))
-    (fp_line (start 1.8 9.4) (end 1.8 -1.8) (layer "F.CrtYd") (width 0.05))
-    (fp_line (start 1.8 -1.8) (end -1.8 -1.8) (layer "F.CrtYd") (width 0.05))
+    (fp_line (start -1.299921 -0.198003) (end -1.299921 7.751997) (layer "B.SilkS") (width 0.12))
+    (fp_line (start 1.3 -0.2) (end 1.3 7.75) (layer "B.SilkS") (width 0.12))
+    (fp_arc (start 1.3 7.75) (mid 0.000999 9.000963) (end -1.299921 7.751997) (layer "B.SilkS") (width 0.12))
+    (fp_arc (start -1.299921 -0.198003) (mid -0.00092 -1.448965) (end 1.3 -0.2) (layer "B.SilkS") (width 0.12))
+    (fp_line (start -1.285344 -0.201036) (end -1.285344 7.75) (layer "F.SilkS") (width 0.12))
+    (fp_line (start 1.314577 -0.199039) (end 1.314577 7.751997) (layer "F.SilkS") (width 0.12))
+    (fp_arc (start -1.285344 -0.201036) (mid 0.015576 -1.45) (end 1.314577 -0.199039) (layer "F.SilkS") (width 0.12))
+    (fp_arc (start 1.314577 7.751997) (mid 0.013657 9.000962) (end -1.285344 7.75) (layer "F.SilkS") (width 0.12))
     (fp_line (start -1.8 -1.8) (end -1.8 9.4) (layer "F.CrtYd") (width 0.05))
     (fp_line (start -1.8 9.4) (end 1.8 9.4) (layer "F.CrtYd") (width 0.05))
+    (fp_line (start 1.8 9.4) (end 1.8 -1.8) (layer "F.CrtYd") (width 0.05))
+    (fp_line (start 1.8 -1.8) (end -1.8 -1.8) (layer "F.CrtYd") (width 0.05))
+    (fp_line (start -0.635 -1.27) (end 1.27 -1.27) (layer "F.Fab") (width 0.1))
+    (fp_line (start -1.27 -0.635) (end -0.635 -1.27) (layer "F.Fab") (width 0.1))
     (fp_line (start -1.27 8.89) (end -1.27 -0.635) (layer "F.Fab") (width 0.1))
     (fp_line (start 1.27 8.89) (end -1.27 8.89) (layer "F.Fab") (width 0.1))
-    (fp_line (start -1.27 -0.635) (end -0.635 -1.27) (layer "F.Fab") (width 0.1))
-    (fp_line (start -0.635 -1.27) (end 1.27 -1.27) (layer "F.Fab") (width 0.1))
     (fp_line (start 1.27 -1.27) (end 1.27 8.89) (layer "F.Fab") (width 0.1))
     (pad "1" thru_hole rect (at 0 0 90) (size 1.7 1.7) (drill 1) (layers *.Cu *.Mask)
@@
   )
   (footprint "kibuzzard-62C19AB4" (layer "F.Cu")
-    (at 152.135 73.87)
+    (at 151.924422 73.86)
     (descr "Converted using: scripting")
     (tags "svg2mod")
@@
   )
   (footprint "kibuzzard-62C19AC2" (layer "B.Cu")
-    (at 152.135 73.87 180)
+    (at 151.95 73.86 180)
     (descr "Converted using: scripting")
     (tags "svg2mod")
@@
       (effects (font (size 1 1) (thickness 0.15)) (justify mirror))
     )
-    (fp_line (start 5.2 9.3) (end 5.2 12.1) (layer "B.SilkS") (width 0.12))
-    (fp_line (start 6.4 -2.8) (end 3.7 -2.8) (layer "B.SilkS") (width 0.12))
-    (fp_line (start -0.6 9.3) (end -0.6 12.1) (layer "B.SilkS") (width 0.12))
-    (fp_line (start 6.4 9.3) (end 6.4 -2.8) (layer "B.SilkS") (width 0.12))
-    (fp_line (start 5.2 12.1) (end -0.6 12.1) (layer "B.SilkS") (width 0.12))
-    (fp_line (start -0.9 -2.8) (end 3.7 -2.8) (layer "B.SilkS") (width 0.12))
-    (fp_line (start -0.9 9.3) (end -0.9 -2.8) (layer "B.SilkS") (width 0.12))
-    (fp_line (start -0.9 9.3) (end -0.6 9.3) (layer "B.SilkS") (width 0.12))
-    (fp_line (start 5.2 9.3) (end 6.4 9.3) (layer "B.SilkS") (width 0.12))
-    (fp_line (start 0.3 9.3) (end -0.9 9.3) (layer "F.SilkS") (width 0.12))
-    (fp_line (start -0.9 -2.8) (end 1.8 -2.8) (layer "F.SilkS") (width 0.12))
-    (fp_line (start 6.4 -2.8) (end 1.8 -2.8) (layer "F.SilkS") (width 0.12))
-    (fp_line (start 0.3 12.1) (end 6.1 12.1) (layer "F.SilkS") (width 0.12))
-    (fp_line (start 6.4 9.3) (end 6.4 -2.8) (layer "F.SilkS") (width 0.12))
-    (fp_line (start -0.9 9.3) (end -0.9 -2.8) (layer "F.SilkS") (width 0.12))
-    (fp_line (start 0.3 9.3) (end 0.3 12.1) (layer "F.SilkS") (width 0.12))
-    (fp_line (start 6.4 9.3) (end 6.1 9.3) (layer "F.SilkS") (width 0.12))
-    (fp_line (start 6.1 9.3) (end 6.1 12.1) (layer "F.SilkS") (width 0.12))
+    (fp_line (start -1.3 12.5) (end -1.3 -3) (layer "B.CrtYd") (width 0.05))
     (fp_line (start -1.3 12.5) (end 6.8 12.5) (layer "B.CrtYd") (width 0.05))
     (fp_line (start 6.8 12.5) (end 6.8 -3) (layer "B.CrtYd") (width 0.05))
     (fp_line (start -1.3 -3) (end 6.8 -3) (layer "B.CrtYd") (width 0.05))
-    (fp_line (start -1.3 12.5) (end -1.3 -3) (layer "B.CrtYd") (width 0.05))
-    (fp_line (start 5.1 9.2) (end 6.3 9.2) (layer "B.Fab") (width 0.1))
-    (fp_line (start 6.3 -2) (end 5.3 -2) (layer "B.Fab") (width 0.1))
+    (fp_line (start -0.5 12) (end 5.1 12) (layer "B.Fab") (width 0.1))
     (fp_line (start -0.8 -2) (end -0.8 9.2) (layer "B.Fab") (width 0.1))
-    (fp_line (start 5.1 12) (end 5.1 9.2) (layer "B.Fab") (width 0.1))
+    (fp_line (start 3.7 -2) (end -0.8 -2) (layer "B.Fab") (width 0.1))
     (fp_line (start -0.8 9.2) (end -0.5 9.2) (layer "B.Fab") (width 0.1))
-    (fp_line (start -0.5 9.2) (end -0.5 12) (layer "B.Fab") (width 0.1))
-    (fp_line (start -0.5 12) (end 5.1 12) (layer "B.Fab") (width 0.1))
     (fp_line (start 6.3 9.2) (end 6.3 -2) (layer "B.Fab") (width 0.1))
-    (fp_line (start 3.7 -2) (end -0.8 -2) (layer "B.Fab") (width 0.1))
+    (fp_line (start 5.1 12) (end 5.1 9.2) (layer "B.Fab") (width 0.1))
+    (fp_line (start 6.3 -2) (end 5.3 -2) (layer "B.Fab") (width 0.1))
+    (fp_line (start 5.1 9.2) (end 6.3 9.2) (layer "B.Fab") (width 0.1))
+    (fp_line (start -0.5 9.2) (end -0.5 12) (layer "B.Fab") (width 0.1))
     (fp_circle (center 0.9 0) (end 1.2 -0.15) (layer "B.Fab") (width 0.12) (fill none))
-    (pad "" np_thru_hole oval (at 2.3 1.6 180) (size 1.5 1.5) (drill oval 1.5) (layers *.Cu *.Mask))
     (pad "" np_thru_hole oval (at 2.3 8.6 180) (size 1.5 1.5) (drill oval 1.5) (layers *.Cu *.Mask))
+    (pad "" np_thru_hole oval (at 2.3 1.6 180) (size 1.5 1.5) (drill oval 1.5) (layers *.Cu *.Mask))
     (pad "R1" thru_hole oval (at 0 4 180) (size 2 1.4) (drill oval 1.2 0.6) (layers *.Cu *.Mask)
       (net 1 "Gnd_l") (pintype "passive"))

Commit message: silkscreen
Parts:
- removed kibuzzard-62BF0E9F: G***, kibuzzard-62BF0E9F
- removed kibuzzard-62BF0EBF: G***, kibuzzard-62BF0EBF
- added kibuzzard-62C547B3: G***, kibuzzard-62C547B3, F.Cu at (160.3, 77.8)
- added kibuzzard-62C5480E: G***, kibuzzard-62C5480E, B.Cu at (160.0, 77.8)
Changed lines of the file:
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@@
     )
   )
+  (footprint "kibuzzard-62C547B3" (layer "F.Cu")
+    (at 160.29 77.85)
+    (descr "Converted using: scripting")
+    (tags "svg2mod")
+    (attr board_only exclude_from_pos_files exclude_from_bom)
+    (fp_text reference "kibuzzard-62C547B3" (at 0 -0.846968) (layer "F.SilkS") hide
+      (effects (font (size 0.000254 0.000254) (thickness 0.000003)))
+    )
+    (fp_text value "G***" (at 0 0.846968) (layer "F.SilkS") hide
+      (effects (font (size 0.000254 0.000254) (thickness 0.000003)))
+    )
+    (fp_poly (pts
+        (xy 2.603911 -0.563919)
+        (xy 2.085338 -0.563919)
+        (xy 2.085338 0.84646)
+        (xy 1.736522 0.84646)
+        (xy 1.736522 -0.563919)
+        (xy 1.224925 -0.563919)
+        (xy 1.224925 -0.84646)
+        (xy 2.603911 -0.84646)
+        (xy 2.603911 -0.563919)
+      ) (layer "F.SilkS") (width 0) (fill solid))
+    (fp_poly (pts
+        (xy -2.255095 0.566245)
+        (xy -1.514442 0.566245)
+        (xy -1.514442 0.84646)
+        (xy -2.603911 0.84646)
+        (xy -2.603911 -0.84646)
+        (xy -2.255095 -0.84646)
+        (xy -2.255095 0.566245)
+      ) (layer "F.SilkS") (width 0) (fill solid))
+    (fp_poly (pts
+        (xy 1.043541 0.154642)
+        (xy 0.373814 0.154642)
+        (xy 0.373814 0.84646)
+        (xy 0.024998 0.84646)
+        (xy 0.024998 -0.84646)
+        (xy 1.127257 -0.84646)
+        (xy 1.127257 -0.563919)
+        (xy 0.373814 -0.563919)
+        (xy 0.373814 -0.126736)
+        (xy 1.043541 -0.126736)
+        (xy 1.043541 0.154642)
+      ) (layer "F.SilkS") (width 0) (fill solid))
+    (fp_poly (pts
+        (xy -0.295912 0.112784)
+        (xy -0.965639 0.112784)
+        (xy -0.965639 0.566245)
+        (xy -0.17964 0.566245)
+        (xy -0.17964 0.84646)
+        (xy -1.314455 0.84646)
+        (xy -1.314455 -0.84646)
+        (xy -0.181966 -0.84646)
+        (xy -0.181966 -0.563919)
+        (xy -0.965639 -0.563919)
+        (xy -0.965639 -0.160455)
+        (xy -0.295912 -0.160455)
+        (xy -0.295912 0.112784)
+      ) (layer "F.SilkS") (width 0) (fill solid))
+  )
   (footprint "Resistor_SMD:R_0402_1005Metric" locked (layer "F.Cu")
     (at 164.055 60.435)
@@
     )
   )
-  (footprint "kibuzzard-62BF0EBF" (layer "F.Cu")
-    (at 144.209006 91.5225)
-    (descr "Converted using: scripting")
-    (tags "svg2mod")
-    (attr board_only exclude_from_pos_files exclude_from_bom)
-    (fp_text reference "kibuzzard-62BF0EBF" (at 0 -1.693428) (layer "F.SilkS") hide
-      (effects (font (size 0.000254 0.000254) (thickness 0.000003)))
-    )
-    (fp_text value "G***" (at 0 1.693428) (layer "F.SilkS") hide
-      (effects (font (size 0.000254 0.000254) (thickness 0.000003)))
-    )
-    (fp_poly (pts
-        (xy -0.391837 1.132489)
-        (xy 1.089468 1.132489)
-        (xy 1.089468 1.69292)
-        (xy -1.089468 1.69292)
-        (xy -1.089468 -1.69292)
-        (xy -0.391837 -1.69292)
-        (xy -0.391837 1.132489)
-      ) (layer "F.SilkS") (width 0) (fill solid))
-  )
   (footprint "local-libraries:R_0402_1005Metric_nolabel" (layer "F.Cu")
     (at 167.05 50.9 90)
@@
       ))
   )
-  (footprint "kibuzzard-62BF0E9F" (layer "B.Cu")
-    (at 143.83 91.5225 180)
+  (footprint "kibuzzard-62C5480E" (layer "B.Cu")
+    (at 159.98 77.81 180)
     (descr "Converted using: scripting")
     (tags "svg2mod")
     (attr board_only exclude_from_pos_files exclude_from_bom)
-    (fp_text reference "kibuzzard-62BF0E9F" (at 0 1.693428) (layer "B.SilkS") hide
+    (fp_text reference "kibuzzard-62C5480E" (at 0 0.870222) (layer "B.SilkS") hide
       (effects (font (size 0.000254 0.000254) (thickness 0.000003)) (justify mirror))
     )
-    (fp_text value "G***" (at 0 -1.693428) (layer "B.SilkS") hide
+    (fp_text value "G***" (at 0 -0.870222) (layer "B.SilkS") hide
       (effects (font (size 0.000254 0.000254) (thickness 0.000003)) (justify mirror))
     )
     (fp_poly (pts
-        (xy -0.065112 -0.453461)
-        (xy -0.620892 0.111621)
-        (xy -0.058136 0.111621)
-        (xy 0.174989 0.145049)
-        (xy 0.348816 0.245334)
-        (xy 0.456949 0.404336)
-        (xy 0.492993 0.613916)
-        (xy 0.458984 0.827856)
-        (xy 0.356955 0.990637)
-        (xy 0.184582 1.093538)
-        (xy -0.060461 1.127838)
-        (xy -0.620892 1.127838)
-        (xy -0.620892 0.111621)
-        (xy -0.065112 -0.453461)
-        (xy -0.620892 -0.453461)
-        (xy -0.620892 -1.69292)
-        (xy -1.318524 -1.69292)
-        (xy -1.318524 1.69292)
-        (xy -0.060461 1.69292)
-        (xy 0.309025 1.663206)
-        (xy 0.617533 1.574064)
-        (xy 0.865063 1.425494)
-        (xy 1.045931 1.222664)
-        (xy 1.154451 0.970742)
-        (xy 1.190625 0.669727)
-        (xy 1.153127 0.352013)
-        (xy 1.040634 0.091855)
-        (xy 0.851983 -0.115981)
-        (xy 0.586011 -0.276727)
-        (xy 1.318524 -1.660364)
-        (xy 1.318524 -1.69292)
-        (xy 0.569733 -1.69292)
-        (xy -0.065112 -0.453461)
+        (xy 1.817331 -0.84646)
+        (xy 1.468515 -0.84646)
+        (xy 1.468515 -0.120923)
+        (xy 0.788324 -0.120923)
+        (xy 0.788324 -0.84646)
+        (xy 0.439508 -0.84646)
+        (xy 0.439508 0.84646)
+        (xy 0.788324 0.84646)
+        (xy 0.788324 0.160455)
+        (xy 1.468515 0.160455)
+        (xy 1.468515 0.84646)
+        (xy 1.817331 0.84646)
+        (xy 1.817331 -0.84646)
+      ) (layer "B.SilkS") (width 0) (fill solid))
+    (fp_poly (pts
+        (xy 3.396304 0.563919)
+        (xy 2.877731 0.563919)
+        (xy 2.877731 -0.84646)
+        (xy 2.528915 -0.84646)
+        (xy 2.528915 0.563919)
+        (xy 2.017319 0.563919)
+        (xy 2.017319 0.84646)
+        (xy 3.396304 0.84646)
+        (xy 3.396304 0.563919)
+      ) (layer "B.SilkS") (width 0) (fill solid))
+    (fp_poly (pts
+        (xy -1.505722 -0.84646)
+        (xy -1.854538 -0.84646)
+        (xy -1.854538 0.84646)
+        (xy -1.505722 0.84646)
+        (xy -1.505722 -0.84646)
+      ) (layer "B.SilkS") (width 0) (fill solid))
+    (fp_poly (pts
+        (xy 0.156967 -0.63252)
+        (xy 0.043311 -0.732659)
+        (xy -0.109296 -0.807509)
+        (xy -0.29068 -0.854163)
+        (xy -0.490668 -0.869714)
+        (xy -0.631163 -0.859056)
+        (xy -0.759644 -0.827081)
+        (xy -0.876109 -0.77379)
+        (xy -1.022903 -0.65621)
+        (xy -1.131908 -0.495319)
+        (xy -1.182228 -0.366515)
+        (xy -1.21304 -0.223501)
+        (xy -1.224344 -0.066275)
+        (xy -1.224344 0.048834)
+        (xy -1.214848 0.210258)
+        (xy -1.186362 0.356567)
+        (xy -1.138884 0.487761)
+        (xy -1.03453 0.651414)
+        (xy -0.892387 0.771465)
+        (xy -0.778893 0.826048)
+        (xy -0.653126 0.858798)
+        (xy -0.515085 0.869714)
+        (xy -0.32892 0.853759)
+        (xy -0.171953 0.805894)
+        (xy -0.044183 0.726118)
+        (xy 0.053614 0.615854)
+        (xy 0.120664 0.476521)
+        (xy 0.156967 0.308121)
+        (xy -0.182547 0.308121)
+        (xy -0.219899 0.433985)
+        (xy -0.285448 0.520898)
+        (xy -0.380064 0.571477)
+        (xy -0.50462 0.588336)
+        (xy -0.661297 0.554908)
+        (xy -0.775534 0.454623)
+        (xy -0.82734 0.351012)
+        (xy -0.858733 0.218462)
+        (xy -0.869714 0.056973)
+        (xy -0.869714 -0.05116)
+        (xy -0.858475 -0.214199)
+        (xy -0.824756 -0.348299)
+        (xy -0.768558 -0.453461)
+        (xy -0.643856 -0.555489)
+        (xy -0.472064 -0.589499)
+        (xy -0.303761 -0.56857)
+        (xy -0.191849 -0.505783)
+        (xy -0.191849 -0.21394)
+        (xy -0.509271 -0.21394)
+        (xy -0.509271 0.043021)
+        (xy 0.156967 0.043021)
+        (xy 0.156967 -0.63252)
+      ) (layer "B.SilkS") (width 0) (fill solid))
+    (fp_poly (pts
+        (xy -2.769598 -0.22673)
+        (xy -3.047488 0.055811)
+        (xy -2.76611 0.055811)
+        (xy -2.649548 0.072525)
+        (xy -2.562634 0.122667)
+        (xy -2.508568 0.202168)
+        (xy -2.490546 0.306958)
+        (xy -2.50755 0.413928)
+        (xy -2.558565 0.495319)
+        (xy -2.644751 0.546769)
+        (xy -2.767273 0.563919)
+        (xy -3.047488 0.563919)
+        (xy -3.047488 0.055811)
+        (xy -2.769598 -0.22673)
+        (xy -3.047488 -0.22673)
+        (xy -3.047488 -0.84646)
+        (xy -3.396304 -0.84646)
+        (xy -3.396304 0.84646)
+        (xy -2.767273 0.84646)
+        (xy -2.58253 0.831603)
+        (xy -2.428276 0.787032)
+        (xy -2.30451 0.712747)
+        (xy -2.214077 0.611332)
+        (xy -2.159816 0.485371)
+        (xy -2.14173 0.334863)
+        (xy -2.160479 0.176007)
+        (xy -2.216725 0.045927)
+        (xy -2.311051 -0.057991)
+        (xy -2.444037 -0.138364)
+        (xy -2.07778 -0.830182)
+        (xy -2.07778 -0.84646)
+        (xy -2.452176 -0.84646)
+        (xy -2.769598 -0.22673)
       ) (layer "B.SilkS") (width 0) (fill solid))
   )
@@
     )
   )
-  (gr_circle (center 144.04 91.4825) (end 146.74 91.4825) (layer "B.SilkS") (width 0.5) (fill none))
   (gr_poly
     (pts
@@
       (xy 151.57 71.0325)
     ) (layer "B.SilkS") (width 0.2) (fill solid))
-  (gr_circle (center 143.94 91.5825) (end 146.64 91.5825) (layer "F.SilkS") (width 0.5) (fill none))
   (gr_poly locked
     (pts

Commit message: jlc parts
Parts:
- D101, D102, D103, D104, D105, D106, D107, D108, D109, D110, D111, D112, D113, D114, D115, D116, D117: footprint local-libraries:D_0402_1005Metric_bkb -> local-libraries:D_1206_handsolder_reversible
Routing:
- net col3_l: track 155.0 -> 159.4 mm
- net col5_l: track 128.2 -> 130.9 mm, vias 2 -> 1
- net col1_l: track 180.3 -> 182.8 mm
- net Net-(D102-Pad2): track 27.0 -> 25.2 mm
- net col2_l: track 135.5 -> 137.1 mm
- net Net-(D106-Pad2): track 26.5 -> 25.3 mm
- net Net-(D101-Pad2): track 26.0 -> 25.2 mm
- net Net-(D108-Pad2): track 26.1 -> 25.3 mm
- net Net-(D115-Pad2): track 25.1 -> 25.9 mm
- net Net-(D113-Pad2): track 24.9 -> 25.6 mm
- net Net-(D112-Pad2): track 26.4 -> 25.7 mm
- net Net-(D103-Pad2): track 27.8 -> 28.5 mm
- net Net-(D114-Pad2): track 26.3 -> 27.0 mm

Commit message: spi breakout
Parts:
- added J107: Conn_01x08_Female, local-libraries:1x08 smd reversible, F.Cu at (143.5, 90.4)
- added kibuzzard-62C55DF6: G***, kibuzzard-62C55DF6, F.Cu at (143.5, 94.2)
- added kibuzzard-62C55DF6: G***, kibuzzard-62C55DF6, B.Cu at (143.5, 94.3)
- moved kibuzzard-61F01A92 57.9 mm to (201.1, 44.1)
Routing:
- net Gnd_l: track 171.8 -> 205.8 mm
- net +3V3: track 120.0 -> 146.8 mm
- net mosi_l: track 42.5 -> 65.7 mm
- net NCS: track 40.3 -> 62.5 mm
- net sda_l: track 53.0 -> 74.4 mm, vias 3 -> 4
- net miso_l: track 39.2 -> 60.1 mm
- net sc_l: track 41.4 -> 59.8 mm
- net scl_l: track 42.2 -> 58.7 mm, vias 4 -> 5
Other:
- board text added: "MISO"
- board text added: "MOSI"
- board text added: "NCS"
- board text added: "SC"
- board text added: "SCL"
- board text added: "SDA"
- board text added: "VCC"
