File: dilemma/0xB2.kicad_sch (KiCad schematic)
At the start: 107 parts, among them J1 USB_C_Receptacle_USB2.0, J101 trackball, J102 Serial, J103 Serial, J104 BATTERY_CONN_DEANS, J105 S3B-PH-SM4-TB(LF)(SN), J106 S3B-PH-SM4-TB(LF)(SN), J107 Conn_01x08_Female, J108 Conn_01x01_Female, J113 Cirque, J5 Conn_01x02, SW1 SW_Push, SW101 SW_Push, SW102 SW_Push, SW103 SW_Push, SW104 SW_Push, SW105 SW_Push, SW106 SW_Push, SW107 SW_Push, SW108 SW_Push, SW109 SW_Push, SW110 SW_SPST, SW111 SW_SPST, SW112 SW_Push, SW113 SW_Push, SW114 SW_Push, SW115 SW_Push, SW116 SW_Push, SW117 SW_Push, SW118 SW_Push, SW119 SW_Push, SW2 SW_Push, U1 RP2040, U2 GD25Q80CEIGR, U3 XC6210B332MR-G, Y1 Crystal_GND24

Commit message: zones
Parts:
- added J109: Conn_01x01_Female, Connector_Wire:SolderWirePad_1x01_SMD_1x2mm, symbol Connector:Conn_01x01_Female
Connections:
- net rgb_l: now also J109.1 (Pin_1)
Changed lines of the file:
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@@
     )
   )
+  (global_label "rgb_l" (shape input) (at 387.985 102.87 180)
+    (effects (font (size 1.27 1.27)) (justify right))
+    (property "Intersheet References" "${INTERSHEET_REFS}" (id 0) (at 300.355 35.56 0)
+      (effects (font (size 1.27 1.27)) hide)
+    )
+  )
   (global_label "Rst_l" (shape input) (at 445.77 111.125 180)
     (effects (font (size 1.27 1.27)) (justify right))
@@
     (pin "1")
   )
+  (symbol (lib_id "Connector:Conn_01x01_Female") (at 393.065 102.87 0) (unit 1)
+    (in_bom yes) (on_board yes) (fields_autoplaced)
+    (property "Reference" "J109" (id 0) (at 394.97 101.5999 0)
+      (effects (font (size 1.27 1.27)) (justify left))
+    )
+    (property "Value" "Conn_01x01_Female" (id 1) (at 394.97 104.1399 0)
+      (effects (font (size 1.27 1.27)) (justify left))
+    )
+    (property "Footprint" "Connector_Wire:SolderWirePad_1x01_SMD_1x2mm" (id 2) (at 393.065 102.87 0)
+      (effects (font (size 1.27 1.27)) hide)
+    )
+    (property "Datasheet" "~" (id 3) (at 393.065 102.87 0)
+      (effects (font (size 1.27 1.27)) hide)
+    )
+    (pin "1")
+  )
   (symbol (lib_id "Device:D") (at 441.96 48.26 180) (unit 1)
     (in_bom yes) (on_board yes)
@@
       (reference "J108") (unit 1) (value "Conn_01x01_Female") (footprint "Connector_Wire:SolderWirePad_1x01_SMD_1x2mm")
     )
+    (path "/db83c478-aecd-42c6-b5c8-ab4611c24929"
+      (reference "J109") (unit 1) (value "Conn_01x01_Female") (footprint "Connector_Wire:SolderWirePad_1x01_SMD_1x2mm")
+    )
     (path "/eeb6b826-bc65-4571-ab3b-1b47a831da34"

Commit message: add license
Other:
- company: plut0nium -> plut0nium x bastardkb x freznel
- title: 0xB2 - Splinky -> Dilemma
Changed lines of the file:
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@@
   (paper "A4")
   (title_block
-    (title "0xB2 - Splinky")
-    (rev "2")
-    (company "plut0nium")
+    (title "Dilemma")
+    (date "2022-07-12")
+    (rev "1")
+    (company "plut0nium x bastardkb x freznel")
+    (comment 1 "Licensed under CERN-OHL-W v2")
   )
   (junction (at 396.24 38.1) (diameter 0) (color 0 0 0 0)
