File: dilemma_assembled_rgb/dilemma.kicad_sch (KiCad schematic)
At the start: 93 parts, among them J1 USB_C_Receptacle_USB2.0, J102 Serial, J105 Conn_01x04_Female, J113 Cirque, J2 Conn_01x03_Female, J5 Conn_01x02, SW1 SW_Push, SW110 SW_SPST, SW2 SW_Push, SW3002 RotaryEncoder_Switch, U1 RP2040, U2 GD25Q80CEIGR, U3 XC6210B332MR-G, U4 USBLC6-2P6, Y1 Crystal_GND24

Commit message: rgb schem work
Parts:
- removed C1, C2: 1µ, Capacitor_SMD:C_0603_1608Metric, symbol Device:C
- removed C10, C11, C12, C13, C14, C7, C8, C9: 100n, Capacitor_SMD:C_0402_1005Metric, symbol Device:C
- removed C3, C4: 15p, Capacitor_SMD:C_0402_1005Metric, symbol Device:C
- removed C5, C6: 1µ, Capacitor_SMD:C_0402_1005Metric, symbol Device:C
- removed D1: LED, LED_SMD:LED_0402_1005Metric, symbol sk6805-ec15:SK6805-hole
- removed D19: NA_SK6805-hole, 0xB2_drawings:LED_SK6805-EC15_hole, symbol sk6805-ec15:SK6805-hole
- removed D2: B5817, Diode_SMD:D_SOD-323, symbol Device:D_Schottky
- removed D3: NA_SK6805-hole, prettylib:LED_SK6805-EC15_1.5x1.5mm_P0.6mm_handsolder, symbol sk6805-ec15:SK6805-hole
- removed F1: Polyfuse, Fuse:Fuse_0603_1608Metric, symbol Device:Polyfuse
- removed FB1: FerriteBead_Small, Inductor_SMD:L_0603_1608Metric, symbol Device:FerriteBead_Small
- removed H102: M4, local-libraries:MountingHole_3mm_Pad_hole, symbol Mechanical:MountingHole_Pad
- removed H103, H109, H110: t, local-libraries:JLC_SMT_Assembly_Hole, symbol Mechanical:MountingHole_Pad
- removed H105, H106, H107, H108: M4, local-libraries:MountingHole_3mm_Pad_Via, symbol Mechanical:MountingHole_Pad
- removed J1: USB_C_Receptacle_USB2.0, 0xLib_USB_Type-C:USB_C_Receptacle_HRO_TYPE-C-31-M-13B, symbol Connector:USB_C_Receptacle_USB2.0
- removed J102: Serial, local-libraries:Jack_3.5mm_PJ320E_Horizontal, symbol Connector:AudioJack4
- removed J105: Conn_01x04_Female, local-libraries:PinHeader_1x04_P2.54mm_Vertical_debug, symbol Connector:Conn_01x04_Female
- removed J113: Cirque, local-libraries:FPC-SMD_FPC05012-09200-.5mm, symbol Connector:Conn_01x14_Female
- removed J2: Conn_01x03_Female, local-libraries:PinHeader_1x03_P2.54mm_Vertical_smd, symbol Connector:Conn_01x03_Female
- removed J5: Conn_01x02, Connector_PinHeader_1.27mm:PinHeader_1x02_P1.27mm_Vertical, symbol Connector_Generic:Conn_01x02
- removed O101: OLED, local-libraries:PinHeader_1x04_P2.54mm_Vertical, symbol Connector_Generic:Conn_01x04
- removed R1, R3, R8: 1k, Resistor_SMD:R_0402_1005Metric, symbol Device:R
- removed R10, R4, R5: 5.1k, Resistor_SMD:R_0402_1005Metric, symbol Device:R
- removed R101: 5.1k, local-libraries:R_0402_1005Metric_nolabel, symbol Device:R
- removed R103, R104: 4.7k, local-libraries:R_0402_1005Metric_nolabel, symbol Device:R
- removed R11, R2, R9: 10k, Resistor_SMD:R_0402_1005Metric, symbol Device:R
- removed R6, R7: 27, Resistor_SMD:R_0402_1005Metric, symbol Device:R
- removed SW1, SW2: SW_Push, Button_Switch_SMD:SW_SPST_CK_KXT3, symbol Switch:SW_Push
- removed SW110: SW_SPST, local-libraries:SW_Push_1P1T_NO_6x6mm_H9.5mm, symbol Switch:SW_SPST
- removed U1: RP2040, 0xLib_Package_DFN_QFN:QFN-56-1EP_7x7mm_P0.4mm_EP3.2x3.2mm, symbol MCU_RaspberryPi_RP2040:RP2040
- removed U2: GD25Q80CEIGR, 0xLib_Package_DFN_QFN:USON-8-1EP_3x2mm_P0.5mm_EP0.25x1.65mm, symbol Memory_Flash:W25Q32JVZP
- removed U3: XC6210B332MR-G, Package_TO_SOT_SMD:SOT-23-5, symbol Regulator_Linear:AP2127K-3.3
- removed U4: USBLC6-2P6, Package_TO_SOT_SMD:SOT-666, symbol Power_Protection:USBLC6-2P6
- removed Y1: Crystal_GND24, Crystal:Crystal_SMD_2520-4Pin_2.5x2.0mm, symbol Device:Crystal_GND24
- added D9: NA_SK6805-hole, 0xB2_drawings:LED_SK6805-EC15_hole, symbol sk6805-ec15:SK6805-hole
- added J1: NA_Conn_01x03_Female, local-libraries:PinHeader_1x03_P2.54mm_Vertical_smd, symbol Connector:Conn_01x03_Female
- H101, H104: value M4 -> NA_M4
- H111: value t -> NA_t
- SW3002: value RotaryEncoder_Switch -> NA_RotaryEncoder_Switch
Connections:
- net +3V3: now also J1.2 (Pin_2)
- net GND: now also J1.1 (Pin_1)
- net RGB: now also J1.3 (Pin_3)
- no-connect marks 24 -> 6
Other:
- note removed: "Assembly holes"
- note removed: "Cirque FPC connector"
- note removed: "Debug breakout"
- note removed: "Decoupling"
- note removed: "ESD protection"
- note removed: "Flash memory"
- note removed: "Handedness"
- note removed: "Indicator & buttons"
- note removed: "MCU"
- note removed: "Mod screws"
- note removed: "OLED connector"
- note removed: "Reset button"
- note removed: "Serial"
- note removed: "USB-C connector"
- note removed: "Voltage regulation"
- note removed: "switch to gnd for left half"
- moved on the sheet: D11, D12, D15, D16, D18, D21, D22, D24, D25, D27, D28, D30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
