File: dilemma_assembled_L/dilemma_L.kicad_sch (KiCad schematic)
At the start: 102 parts, among them J1 USB_C_Receptacle_USB2.0, J102 NA_serial, J105 NA_Conn_01x04_Female, J113 Cirque, J2 NA_Conn_01x03_Female, J3 NA_GC9A01, J4 Conn_01x05, J5 NA_Conn_01x02, SW1 SW_Push, SW101 NA_SW_Push, SW102 NA_SW_Push, SW103 NA_SW_Push, SW104 NA_SW_Push, SW105 NA_SW_Push, SW106 NA_SW_Push, SW107 NA_SW_Push, SW108 NA_SW_Push, SW109 NA_SW_Push, SW112 NA_SW_Push, SW113 NA_SW_Push, SW114 NA_SW_Push, SW115 NA_SW_Push, SW116 NA_SW_Push, SW117 NA_SW_Push, SW118 NA_SW_Push, SW119 NA_SW_Push, SW3001 NA_SW_Push, SW3002 NA_RotaryEncoder_Switch, U1 RP2040, U2 W25Q128JVS, U3 XC6210B332MR-G, U4 USBLC6-2P6, Y1 Crystal_GND24

Commit message: update to left
Connections:
- net SERIAL_L: no longer U1.3 (GPIO1)
- net ENC_PIN1 renamed ENC_PIN1_L
- net ENC_PIN2 renamed ENC_PIN2_L
- net HAND renamed HAND_L
- net IO18 renamed IO18_L
- net M_COL5 renamed M_COL5_L
- net M_ROW1 renamed M_ROW1_L
- net M_ROW4 renamed M_ROW4_L
- net NCS renamed NCS_L
- net QSPI_D0 renamed QSPI_D0_L
- net QSPI_D1 renamed QSPI_D1_L
- net QSPI_D2 renamed QSPI_D2_L
- net QSPI_D3 renamed QSPI_D3_L
- net QSPI_SCLK renamed QSPI_SCLK_L
- net QSPI_~{CS} renamed QSPI_~{CS}_L
- net SWCLK renamed SWCLK_L
- net SWD renamed SWD_L
- net encoder_diode renamed encoder_diode_L
- net ~{RESET} renamed ~{RESET_L}
- new net SERIAL_L_L: U1.3 (GPIO1)

Commit message: more
Connections:
- net D+ renamed D+_L
- net D- renamed D-_L
- net LED renamed LED_L
- net MISO renamed MISO_L
- net MOSI renamed MOSI_L
- net SCLK renamed SCLK_L
- net VBUS_DET renamed VBUS_DET_L
Changed lines of the file:
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@@
     (effects (font (size 1.27 1.27)) (justify left bottom))
   )
-  (label "SCLK" (at 191.77 114.3 180)
+  (label "SCLK_L" (at 191.77 114.3 180)
     (effects (font (size 1.27 1.27)) (justify right bottom))
   )
@@
     (effects (font (size 1.27 1.27)) (justify right bottom))
   )
-  (label "LED" (at 191.77 101.6 180)
+  (label "LED_L" (at 191.77 101.6 180)
     (effects (font (size 1.27 1.27)) (justify right bottom))
   )
-  (label "VBUS_DET" (at 195.58 106.68 180)
+  (label "VBUS_DET_L" (at 195.58 106.68 180)
     (effects (font (size 1.27 1.27)) (justify right bottom))
   )
-  (label "MOSI" (at 191.77 116.84 180)
+  (label "MOSI_L" (at 191.77 116.84 180)
     (effects (font (size 1.27 1.27)) (justify right bottom))
   )
-  (label "D-" (at 111.76 83.82 0)
+  (label "D-_L" (at 111.76 83.82 0)
     (effects (font (size 1.27 1.27)) (justify left bottom))
   )
@@
     (effects (font (size 1.27 1.27)) (justify left bottom))
   )
-  (label "SCLK" (at 296.545 62.23 180)
+  (label "SCLK_L" (at 296.545 62.23 180)
     (effects (font (size 1.27 1.27)) (justify right bottom))
   )
@@
     (effects (font (size 1.27 1.27)) (justify right bottom))
   )
-  (label "D-" (at 192.405 225.425 180)
+  (label "D-_L" (at 192.405 225.425 180)
     (effects (font (size 1.27 1.27)) (justify right bottom))
   )
-  (label "D-" (at 192.405 220.345 180)
+  (label "D-_L" (at 192.405 220.345 180)
     (effects (font (size 1.27 1.27)) (justify right bottom))
   )
@@
     (effects (font (size 1.27 1.27)) (justify left bottom))
   )
-  (label "D+" (at 212.725 220.345 0)
+  (label "D+_L" (at 212.725 220.345 0)
     (effects (font (size 1.27 1.27)) (justify left bottom))
   )
@@
     (effects (font (size 1.27 1.27)) (justify right bottom))
   )
-  (label "D+" (at 111.76 81.28 0)
+  (label "D+_L" (at 111.76 81.28 0)
     (effects (font (size 1.27 1.27)) (justify left bottom))
   )
-  (label "D-" (at 60.325 52.07 180)
+  (label "D-_L" (at 60.325 52.07 180)
     (effects (font (size 1.27 1.27)) (justify right bottom))
   )
-  (label "LED" (at 24.765 160.02 270)
+  (label "LED_L" (at 24.765 160.02 270)
     (effects (font (size 1.27 1.27)) (justify right bottom))
   )
-  (label "MOSI" (at 342.265 48.26 180)
+  (label "MOSI_L" (at 342.265 48.26 180)
     (effects (font (size 1.27 1.27)) (justify right bottom))
   )
-  (label "MOSI" (at 296.545 64.77 180)
+  (label "MOSI_L" (at 296.545 64.77 180)
     (effects (font (size 1.27 1.27)) (justify right bottom))
   )
@@
     (effects (font (size 1.27 1.27)) (justify right bottom))
   )
-  (label "MISO" (at 191.77 109.22 180)
+  (label "MISO_L" (at 191.77 109.22 180)
     (effects (font (size 1.27 1.27)) (justify right bottom))
   )
-  (label "SCLK" (at 342.265 58.42 180)
+  (label "SCLK_L" (at 342.265 58.42 180)
     (effects (font (size 1.27 1.27)) (justify right bottom))
   )
@@
     (effects (font (size 1.27 1.27)) (justify right bottom))
   )
-  (label "MISO" (at 342.265 55.88 180)
+  (label "MISO_L" (at 342.265 55.88 180)
     (effects (font (size 1.27 1.27)) (justify right bottom))
   )
@@
     (effects (font (size 1.27 1.27)) (justify right bottom))
   )
-  (label "D+" (at 60.325 54.61 180)
+  (label "D+_L" (at 60.325 54.61 180)
     (effects (font (size 1.27 1.27)) (justify right bottom))
   )
@@
     (effects (font (size 1.27 1.27)) (justify left bottom))
   )
-  (label "D+" (at 212.725 225.425 0)
+  (label "D+_L" (at 212.725 225.425 0)
     (effects (font (size 1.27 1.27)) (justify left bottom))
   )

Commit message: 3V
Connections:
- net SERIAL_L_L is gone; now on net SERIAL_L: U1.3 (GPIO1)
- net +3V3 renamed +3V3_L
- net +5V renamed +5V_L
- net VBUS renamed VBUS_L

Commit message: gnd
Connections:
- net GND renamed GND_L

Commit message: 1v1
Connections:
- net +1V1 renamed +1V1_L
Other:
- moved on the sheet: O101
Changed lines of the file:
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@@
     (stroke (width 0) (type default) (color 0 0 0 0))
   )
-  (wire (pts (xy 245.745 33.655) (xy 254 33.655))
+  (wire (pts (xy 222.25 34.29) (xy 230.505 34.29))
     (stroke (width 0) (type default) (color 0 0 0 0))
   )
@@
     )
   )
-  (global_label "SDA_L" (shape input) (at 254 38.735 180)
+  (global_label "SDA_L" (shape input) (at 230.505 39.37 180)
     (effects (font (size 1.27 1.27)) (justify right))
-    (property "Intersheet References" "${INTERSHEET_REFS}" (id 0) (at 224.79 -15.875 0)
+    (property "Intersheet References" "${INTERSHEET_REFS}" (id 0) (at 201.295 -15.24 0)
       (effects (font (size 1.27 1.27)) hide)
     )
@@
     )
   )
-  (global_label "SCL_L" (shape input) (at 254 36.195 180)
+  (global_label "SCL_L" (shape input) (at 230.505 36.83 180)
     (effects (font (size 1.27 1.27)) (justify right))
-    (property "Intersheet References" "${INTERSHEET_REFS}" (id 0) (at 224.79 -18.415 0)
+    (property "Intersheet References" "${INTERSHEET_REFS}" (id 0) (at 201.295 -17.78 0)
       (effects (font (size 1.27 1.27)) hide)
     )
@@
     (pin "6")
   )
-  (symbol (lib_id "power_L:GND_L") (at 254 31.115 270) (unit 1)
+  (symbol (lib_id "power_L:GND_L") (at 230.505 31.75 270) (unit 1)
     (in_bom yes) (on_board yes) (fields_autoplaced)
-    (property "Reference" "#PWR?" (id 0) (at 247.65 31.115 0)
+    (property "Reference" "#PWR?" (id 0) (at 224.155 31.75 0)
       (effects (font (size 1.27 1.27)) hide)
     )
-    (property "Value" "GND_L" (id 1) (at 255.27 31.1149 90)
+    (property "Value" "GND_L" (id 1) (at 231.775 31.7499 90)
       (effects (font (size 1.27 1.27)) (justify left))
     )
-    (property "Footprint" "" (id 2) (at 254 31.115 0)
+    (property "Footprint" "" (id 2) (at 230.505 31.75 0)
       (effects (font (size 1.27 1.27)) hide)
     )
-    (property "Datasheet" "" (id 3) (at 254 31.115 0)
+    (property "Datasheet" "" (id 3) (at 230.505 31.75 0)
       (effects (font (size 1.27 1.27)) hide)
     )
@@
     (pin "S1")
   )
-  (symbol (lib_id "power_L:+3V3_L") (at 245.745 33.655 0) (unit 1)
+  (symbol (lib_id "power_L:+1V1_L") (at 101.6 173.99 0) (unit 1)
     (in_bom yes) (on_board yes) (fields_autoplaced)
-    (property "Reference" "#PWR?" (id 0) (at 245.745 37.465 0)
+    (property "Reference" "#PWR?" (id 0) (at 101.6 177.8 0)
       (effects (font (size 1.27 1.27)) hide)
     )
-    (property "Value" "+3V3_L" (id 1) (at 245.745 28.575 0))
-    (property "Footprint" "" (id 2) (at 245.745 33.655 0)
+    (property "Value" "+1V1_L" (id 1) (at 101.6 168.275 0))
+    (property "Footprint" "" (id 2) (at 101.6 173.99 0)
+      (effects (font (size 1.27 1.27)) hide)
+    )
+    (property "Datasheet" "" (id 3) (at 101.6 173.99 0)
+      (effects (font (size 1.27 1.27)) hide)
+    )
+    (pin "1")
+  )
+  (symbol (lib_id "power_L:+3V3_L") (at 222.25 34.29 0) (unit 1)
+    (in_bom yes) (on_board yes) (fields_autoplaced)
+    (property "Reference" "#PWR?" (id 0) (at 222.25 38.1 0)
       (effects (font (size 1.27 1.27)) hide)
     )
-    (property "Datasheet" "" (id 3) (at 245.745 33.655 0)
+    (property "Value" "+3V3_L" (id 1) (at 222.25 29.21 0))
+    (property "Footprint" "" (id 2) (at 222.25 34.29 0)
+      (effects (font (size 1.27 1.27)) hide)
+    )
+    (property "Datasheet" "" (id 3) (at 222.25 34.29 0)
       (effects (font (size 1.27 1.27)) hide)
     )
@@
     (pin "1")
   )
-  (symbol (lib_id "Connector_Generic:Conn_01x04") (at 259.08 33.655 0) (unit 1)
+  (symbol (lib_id "Connector_Generic:Conn_01x04") (at 235.585 34.29 0) (unit 1)
     (in_bom yes) (on_board yes)
-    (property "Reference" "O101" (id 0) (at 262.89 32.8445 0))
-    (property "Value" "NA_OLED" (id 1) (at 264.16 35.3845 0))
-    (property "Footprint" "local-libraries:PinHeader_1x04_P2.54mm_Vertical" (id 2) (at 259.08 33.655 0)
+    (property "Reference" "O101" (id 0) (at 239.395 33.4795 0))
+    (property "Value" "NA_OLED" (id 1) (at 240.665 36.0195 0))
+    (property "Footprint" "local-libraries:PinHeader_1x04_P2.54mm_Vertical" (id 2) (at 235.585 34.29 0)
       (effects (font (size 1.27 1.27)) hide)
     )
-    (property "Datasheet" "" (id 3) (at 259.08 33.655 0)
+    (property "Datasheet" "" (id 3) (at 235.585 34.29 0)
       (effects (font (size 1.27 1.27)) hide)
     )
@@
     (pin "4")
   )
-  (symbol (lib_id "power:+1V1") (at 101.6 173.99 0) (unit 1)
-    (in_bom yes) (on_board yes)
-    (property "Reference" "#PWR017" (id 0) (at 101.6 177.8 0)
-      (effects (font (size 1.27 1.27)) hide)
-    )
-    (property "Value" "+1V1" (id 1) (at 101.6 170.18 0))
-    (property "Footprint" "" (id 2) (at 101.6 173.99 0)
-      (effects (font (size 1.27 1.27)) hide)
-    )
-    (property "Datasheet" "" (id 3) (at 101.6 173.99 0)
-      (effects (font (size 1.27 1.27)) hide)
-    )
-    (pin "1")
-  )
   (symbol (lib_id "kbd:IPS_LCD__gc9a01_240X240") (at 283.845 64.77 0) (mirror y) (unit 1)
     (in_bom no) (on_board yes)
@@
     (pin "1")
   )
-  (symbol (lib_id "power:+1V1") (at 91.44 173.99 0) (unit 1)
-    (in_bom yes) (on_board yes)
-    (property "Reference" "#PWR014" (id 0) (at 91.44 177.8 0)
-      (effects (font (size 1.27 1.27)) hide)
-    )
-    (property "Value" "+1V1" (id 1) (at 91.44 170.18 0))
-    (property "Footprint" "" (id 2) (at 91.44 173.99 0)
-      (effects (font (size 1.27 1.27)) hide)
-    )
-    (property "Datasheet" "" (id 3) (at 91.44 173.99 0)
-      (effects (font (size 1.27 1.27)) hide)
-    )
-    (pin "1")
-  )
   (symbol (lib_id "power_L:+3V3_L") (at 134.62 36.83 0) (unit 1)
     (in_bom yes) (on_board yes) (fields_autoplaced)
@@
     (pin "2")
   )
+  (symbol (lib_id "power_L:+1V1_L") (at 91.44 173.99 0) (unit 1)
+    (in_bom yes) (on_board yes) (fields_autoplaced)
+    (property "Reference" "#PWR?" (id 0) (at 91.44 177.8 0)
+      (effects (font (size 1.27 1.27)) hide)
+    )
+    (property "Value" "+1V1_L" (id 1) (at 91.44 168.275 0))
+    (property "Footprint" "" (id 2) (at 91.44 173.99 0)
+      (effects (font (size 1.27 1.27)) hide)
+    )
+    (property "Datasheet" "" (id 3) (at 91.44 173.99 0)
+      (effects (font (size 1.27 1.27)) hide)
+    )
+    (pin "1")
+  )
   (symbol (lib_id "Device:C") (at 58.42 121.92 0) (unit 1)
     (in_bom yes) (on_board yes)
@@
     (pin "2")
   )
-  (symbol (lib_id "power:+1V1") (at 143.51 36.83 0) (unit 1)
-    (in_bom yes) (on_board yes)
-    (property "Reference" "#PWR022" (id 0) (at 143.51 40.64 0)
-      (effects (font (size 1.27 1.27)) hide)
-    )
-    (property "Value" "+1V1" (id 1) (at 143.51 33.02 0))
-    (property "Footprint" "" (id 2) (at 143.51 36.83 0)
-      (effects (font (size 1.27 1.27)) hide)
-    )
-    (property "Datasheet" "" (id 3) (at 143.51 36.83 0)
-      (effects (font (size 1.27 1.27)) hide)
-    )
-    (pin "1")
-  )
   (symbol (lib_id "power_L:+3V3_L") (at 58.42 109.22 0) (unit 1)
     (in_bom yes) (on_board yes) (fields_autoplaced)
@@
     (pin "1")
   )
+  (symbol (lib_id "power_L:+1V1_L") (at 143.51 36.83 0) (unit 1)
+    (in_bom yes) (on_board yes) (fields_autoplaced)
+    (property "Reference" "#PWR?" (id 0) (at 143.51 40.64 0)
+      (effects (font (size 1.27 1.27)) hide)
+    )
+    (property "Value" "+1V1_L" (id 1) (at 143.51 31.115 0))
+    (property "Footprint" "" (id 2) (at 143.51 36.83 0)
+      (effects (font (size 1.27 1.27)) hide)
+    )
+    (property "Datasheet" "" (id 3) (at 143.51 36.83 0)
+      (effects (font (size 1.27 1.27)) hide)
+    )
+    (pin "1")
+  )
   (symbol (lib_id "sk6805-ec15:SK6805-EC15") (at 546.735 55.88 0) (unit 1)
     (in_bom yes) (on_board yes)
@@
   )
   (symbol_instances
-    (path "/76222eb4-6e0b-40db-aaf4-d0a656e3dbbf"
-      (reference "#PWR014") (unit 1) (value "+1V1") (footprint "")
-    )
-    (path "/6d349fd3-d511-4353-8196-789d1d4f0da4"
-      (reference "#PWR017") (unit 1) (value "+1V1") (footprint "")
-    )
-    (path "/8820d009-4e9a-4453-93b5-85f20fb45b3e"
-      (reference "#PWR022") (unit 1) (value "+1V1") (footprint "")
-    )
     (path "/00a46835-9a8a-491b-9dea-492129e7e807"
       (reference "#PWR?") (unit 1) (value "GND_L") (footprint "")
@@
       (reference "#PWR?") (unit 1) (value "+3V3_L") (footprint "")
     )
+    (path "/61a60e83-845c-4cc9-b932-4760b096cce3"
+      (reference "#PWR?") (unit 1) (value "+1V1_L") (footprint "")
+    )
     (path "/62dad301-a744-4baf-8a77-0500dd271832"
       (reference "#PWR?") (unit 1) (value "+3V3_L") (footprint "")
@@
       (reference "#PWR?") (unit 1) (value "+3V3_L") (footprint "")
     )
+    (path "/858ea5d1-5538-4a90-b6ad-6a4970125658"
+      (reference "#PWR?") (unit 1) (value "+1V1_L") (footprint "")
+    )
     (path "/88f81e81-8cc8-4c7d-adef-999d10589a7b"
       (reference "#PWR?") (unit 1) (value "+3V3_L") (footprint "")
@@
       (reference "#PWR?") (unit 1) (value "GND_L") (footprint "")
     )
+    (path "/cf8d84c2-6ff6-48b8-a6e4-045e90e1fdb8"
+      (reference "#PWR?") (unit 1) (value "+1V1_L") (footprint "")
+    )
     (path "/dcc568a5-dad6-477b-969f-341b34919e1a"

Commit message: annotate from 5000
Parts:
- renumbered C1 to C5001, C2 to C5002, C5 to C5003, C6 to C5004, C3 to C5005, C7 to C5006, C8 to C5007, C4 to C5008, C9 to C5009, C10 to C5010, C11 to C5011, C12 to C5012, C13 to C5013, C14 to C5014, D1 to D5001, D30 to D5002, D35 to D5003, D2 to D5004, D31 to D5005, D36 to D5006, D32 to D5007, D37 to D5008, D112 to D5009, D33 to D5010, D115 to D5011, D34 to D5012, D3 to D5013, D4 to D5014, D5 to D5015, D7 to D5016, D8 to D5017, D11 to D5018, D12 to D5019, D15 to D5020, D9 to D5021, D18 to D5022, D16 to D5023, D21 to D5024, D19 to D5025, D24 to D5026, D22 to D5027, D27 to D5028, D25 to D5029, D28 to D5030, F1 to F5001, FB1 to FB5001, H101 to H5001, H102 to H5002, H104 to H5003, H105 to H5004, H106 to H5005, H107 to H5006, H108 to H5007, H111 to H5008, J1 to J5001, J5 to J5002, J102 to J5003, J3 to J5004, J105 to J5005, J2 to J5006, J113 to J5007, J4 to J5008, O101 to O5001, R1 to R5001, R2 to R5002, R3 to R5003, R5 to R5004, R4 to R5005, R6 to R5006, R7 to R5007, R8 to R5008, R10 to R5009, R11 to R5010, R9 to R5011, R101 to R5012, R103 to R5013, R104 to R5014, SW1 to SW5001, SW101 to SW5002, SW102 to SW5003, SW103 to SW5004, SW118 to SW5005, SW104 to SW5006, SW105 to SW5007, SW106 to SW5008, SW119 to SW5009, SW107 to SW5010, SW108 to SW5011, SW109 to SW5012, SW3001 to SW5013, SW112 to SW5014, SW113 to SW5015, SW114 to SW5016, SW115 to SW5017, SW116 to SW5018, SW117 to SW5019, SW3002 to SW5020, U3 to U5001, U1 to U5002, U4 to U5003, U2 to U5004, Y1 to Y5001
