File: dilemma_assembled/dilemma.kicad_sch (KiCad schematic)
At the start: 102 parts, among them J1 USB_C_Receptacle_USB2.0, J102 NA_serial, J105 NA_Conn_01x04_Female, J113 Cirque, J2 NA_Conn_01x03_Female, J3 NA_GC9A01, J4 Conn_01x05, J5 NA_Conn_01x02, SW1 SW_Push, SW101 NA_SW_Push, SW102 NA_SW_Push, SW103 NA_SW_Push, SW104 NA_SW_Push, SW105 NA_SW_Push, SW106 NA_SW_Push, SW107 NA_SW_Push, SW108 NA_SW_Push, SW109 NA_SW_Push, SW112 NA_SW_Push, SW113 NA_SW_Push, SW114 NA_SW_Push, SW115 NA_SW_Push, SW116 NA_SW_Push, SW117 NA_SW_Push, SW118 NA_SW_Push, SW119 NA_SW_Push, SW3001 NA_SW_Push, SW3002 NA_RotaryEncoder_Switch, U1 RP2040, U2 W25Q128JVS, U3 XC6210B332MR-G, U4 USBLC6-2P6, Y1 Crystal_GND24

Commit message: import to right
Parts:
- added C5001, C5002: 1µ, Capacitor_SMD:C_0603_1608Metric, symbol Device:C
- added C5003, C5004: 1µ, Capacitor_SMD:C_0402_1005Metric, symbol Device:C
- added C5005, C5008: 15p, Capacitor_SMD:C_0402_1005Metric, symbol Device:C
- added C5006, C5007, C5009, C5010, C5011, C5012, C5013, C5014: 100n, Capacitor_SMD:C_0402_1005Metric, symbol Device:C
- added D5001: LED, LED_SMD:LED_0402_1005Metric, symbol Device:LED
- added D5002, D5003, D5005, D5006, D5007, D5008, D5010, D5012: D_CC, local-libraries:SOT-323_SC-70, symbol Device:D_Dual_CommonCathode_AAK
- added D5004: B5817, Diode_SMD:D_SOD-323, symbol Device:D_Schottky
- added D5009, D5011: D, local-libraries:D_SOD-323, symbol Device:D
- added D5013, D5014, D5015, D5016, D5017, D5018, D5019, D5020, D5021, D5022, D5023, D5024, D5025, D5026, D5027, D5028, D5029, D5030: SK6805-EC15, 0xB2_drawings:LED_SK6805-EC15_1.5x1.5mm_P0.6mm_handsolder(1), symbol sk6805-ec15:SK6805-EC15
- added F5001: Polyfuse, Fuse:Fuse_0603_1608Metric, symbol Device:Polyfuse
- added FB5001: FerriteBead_Small, Inductor_SMD:L_0603_1608Metric, symbol Device:FerriteBead_Small
- added H5001, H5002, H5003, H5004, H5005, H5006, H5007: NA_M4, local-libraries:MountingHole_3mm_Pad_Via, symbol Mechanical:MountingHole_Pad
- added H5008: NA_Mount, local-libraries:Tenting_Puck, symbol Mechanical:MountingHole_Pad
- added J5001: USB_C_Receptacle_USB2.0, 0xLib_USB_Type-C:USB_C_Receptacle_HRO_TYPE-C-31-M-13B, symbol Connector:USB_C_Receptacle_USB2.0
- added J5002: NA_Conn_01x02, Connector_PinHeader_1.27mm:PinHeader_1x02_P1.27mm_Vertical, symbol Connector_Generic:Conn_01x02
- added J5003: NA_serial, local-libraries:Jack_3.5mm_PJ320E_Horizontal, symbol Connector:AudioJack4
- added J5004: NA_GC9A01, local-libraries:PinHeader_1x07_P2.54mm_Vertical, symbol kbd:IPS_LCD__gc9a01_240X240
- added J5005: NA_Conn_01x04_Female, local-libraries:PinHeader_1x04_P2.54mm_Vertical_debug, symbol Connector:Conn_01x04_Female
- added J5006: NA_Conn_01x03_Female, local-libraries:PinHeader_1x03_P2.54mm_Vertical_smd, symbol Connector:Conn_01x03_Female
- added J5007: Cirque, local-libraries:FPC-SMD_FPC05012-09200-.5mm, symbol Connector:Conn_01x14_Female
- added J5008: Conn_01x05, local-libraries:PinHeader_1x05_P1.27mm_Vertical_SMD, symbol Connector_Generic:Conn_01x05
- added O5001: NA_OLED, local-libraries:PinHeader_1x04_P2.54mm_Vertical, symbol Connector_Generic:Conn_01x04
- added R5001, R5003, R5008: 1k, Resistor_SMD:R_0402_1005Metric, symbol Device:R
- added R5002, R5010, R5011: 10k, Resistor_SMD:R_0402_1005Metric, symbol Device:R
- added R5004, R5005, R5009: 5.1k, Resistor_SMD:R_0402_1005Metric, symbol Device:R
- added R5006, R5007: 27, Resistor_SMD:R_0402_1005Metric, symbol Device:R
- added R5012: 5.1k, local-libraries:R_0402_1005Metric_nolabel, symbol Device:R
- added R5013, R5014: 4.7k, local-libraries:R_0402_1005Metric_nolabel, symbol Device:R
- added SW5001: SW_Push, Button_Switch_SMD:SW_SPST_CK_KXT3, symbol Switch:SW_Push
- added SW5002, SW5003, SW5004, SW5005, SW5006, SW5007, SW5008, SW5009, SW5010, SW5011, SW5012, SW5013, SW5014, SW5015, SW5016, SW5017, SW5018, SW5019: NA_SW_Push, local-libraries:SW_MX_choc, symbol Switch:SW_Push
- added SW5020: NA_RotaryEncoder_Switch, local-libraries:RotaryEncoder_Alps_EC11E-Switch_Vertical_H20mm_roundholes, symbol Device:RotaryEncoder_Switch
- added U5001: XC6210B332MR-G, Package_TO_SOT_SMD:SOT-23-5, symbol Regulator_Linear:AP2127K-3.3
- added U5002: RP2040, 0xLib_Package_DFN_QFN:QFN-56-1EP_7x7mm_P0.4mm_EP3.2x3.2mm, symbol MCU_RaspberryPi_RP2040:RP2040
- added U5003: USBLC6-2P6, Package_TO_SOT_SMD:SOT-666, symbol Power_Protection:USBLC6-2P6
- added U5004: W25Q128JVS, drawings:W25Q128JVPIQ, symbol Memory_Flash:W25Q128JVS
- added Y5001: Crystal_GND24, Crystal:Crystal_SMD_2520-4Pin_2.5x2.0mm, symbol Device:Crystal_GND24
Connections:
- new net: D5002.1 (A), SW5003.2
- new net: D5009.2 (A), SW5016.2
- new net: D5019.3 (DOUT), D5021.1 (DIN)
- new net: D5021.3 (DOUT), D5023.1 (DIN)
- new net: D5024.3 (DOUT), D5026.1 (DIN)
- new net: D5026.3 (DOUT), D5028.1 (DIN)
- new net: J5002.2 (Pin_2), R5003.1
- new net: D5007.1 (A), SW5011.2
- new net: D5007.2 (A), SW5010.2
- new net: D5008.2 (A), SW5012.2
- new net: D5027.3 (DOUT), D5029.1 (DIN)
- new net: D5029.3 (DOUT), D5030.1 (DIN)
- new net: D5003.1 (A), SW5005.2
- new net: D5003.2 (A), SW5004.2
- new net: D5014.1 (DIN), D5028.3 (DOUT)
- new net: R5006.2, U5002.47 (USB_DP)
- new net: D5013.3 (DOUT), D5016.1 (DIN)
- new net: D5006.1 (A), SW5009.2
- new net: D5012.1 (A), SW5018.2
- new net: D5012.2 (A), SW5017.2
- new net: D5015.1 (DIN), D5030.3 (DOUT)
- new net: D5001.1 (K), R5001.2
- new net: D5022.3 (DOUT), D5024.1 (DIN)
- new net: D5018.3 (DOUT), D5020.1 (DIN)
- new net: D5020.3 (DOUT), D5022.1 (DIN)
- new net: D5004.2 (A), F5001.2
- new net: J5001.A5 (CC1), R5005.1
- new net: J5001.B5 (CC2), R5004.1
- new net: FB5001.2, J5001.S1 (SHIELD)
- new net: D5002.2 (A), SW5002.2
- new net: D5010.2 (A), SW5014.2
- new net: D5011.2 (A), SW5019.2
- new net: C5005.1, U5002.20 (XIN), Y5001.1
- new net: R5008.2, U5002.21 (XOUT)
- new net: R5007.2, U5002.46 (USB_DM)
- new net: D5025.3 (DOUT), D5027.1 (DIN)
- new net: D5016.3 (DOUT), D5018.1 (DIN)
- new net: D5023.3 (DOUT), D5025.1 (DIN)
- new net: D5005.1 (A), SW5007.2
- new net: D5005.2 (A), SW5006.2
- new net: C5008.1, R5008.1, Y5001.3
- new net: D5014.3 (DOUT), D5017.1 (DIN)
- new net: D5017.3 (DOUT), D5019.1 (DIN)
- new net: D5010.1 (A), SW5015.2
- new net: D5006.2 (A), SW5008.2
- new net +1V1_L: C5004.1, C5006.1, C5007.1, U5002.23 (DVDD), U5002.45 (VREG_VOUT), U5002.50 (DVDD)
- new net +3V3_L: C5002.1, C5003.1, C5009.1, C5010.1, C5011.1, C5012.1, C5013.1, C5014.1, D5013.2 (VDD), D5014.2 (VDD), D5015.2 (VDD), D5016.2 (VDD), D5017.2 (VDD), D5018.2 (VDD), D5019.2 (VDD), D5020.2 (VDD), D5021.2 (VDD), D5022.2 (VDD), D5023.2 (VDD), D5024.2 (VDD), D5025.2 (VDD), D5026.2 (VDD), D5027.2 (VDD), D5028.2 (VDD), D5029.2 (VDD), D5030.2 (VDD), J5003.T, J5004.1 (VCC), J5005.1 (Pin_1), J5006.2 (Pin_2), J5007.12 (Pin_12), J5008.1 (Pin_1), O5001.2 (Pin_2), R5002.2, R5011.2, R5012.2, R5013.2, R5014.1, U5001.5 (VOUT), U5002.1 (IOVDD), U5002.10 (IOVDD), U5002.22 (IOVDD), U5002.33 (IOVDD), U5002.42 (IOVDD), U5002.43 (ADC_AVDD), U5002.44 (VREG_IN), U5002.48 (USB_VDD), U5002.49 (IOVDD), U5004.8 (VCC)
- new net +5V_L: C5001.1, D5004.1 (K), U5001.1 (VIN), U5001.3 (EN)
- new net D+_L: J5001.A6 (D+), J5001.B6 (D+), R5006.1, U5003.3 (I/O2), U5003.4 (I/O2)
- new net D-_L: J5001.A7 (D-), J5001.B7 (D-), R5007.1, U5003.1 (I/O1), U5003.6 (I/O1)
- new net ENC_PIN1_L: SW5020.B, U5002.36 (GPIO24)
- new net ENC_PIN2_L: SW5020.A, U5002.37 (GPIO25)
- new net GND_L: C5001.2, C5002.2, C5003.2, C5004.2, C5005.2, C5006.2, C5007.2, C5008.2, C5009.2, C5010.2, C5011.2, C5012.2, C5013.2, C5014.2, D5013.4 (GND), D5014.4 (GND), D5015.4 (GND), D5016.4 (GND), D5017.4 (GND), D5018.4 (GND), D5019.4 (GND), D5020.4 (GND), D5021.4 (GND), D5022.4 (GND), D5023.4 (GND), D5024.4 (GND), D5025.4 (GND), D5026.4 (GND), D5027.4 (GND), D5028.4 (GND), D5029.4 (GND), D5030.4 (GND), FB5001.1, H5001.1, H5002.1, H5003.1, H5004.1, H5005.1, H5006.1, H5007.1, H5008.1, J5001.A1 (GND), J5001.A12 (GND), J5001.B1 (GND), J5001.B12 (GND), J5002.1 (Pin_1), J5003.R1, J5004.2 (GND), J5005.4 (Pin_4), J5006.1 (Pin_1), J5007.11 (Pin_11), J5008.5 (Pin_5), O5001.1 (Pin_1), R5001.1, R5004.2, R5005.2, R5010.1, SW5001.1, SW5020.C, U5001.2 (GND), U5002.19 (TESTEN), U5002.57 (GND), U5003.2 (GND), U5004.4 (GND), Y5001.2, Y5001.4
- new net HAND_L: R5012.1, U5002.41 (GPIO29_ADC3)
- new net IO16_L: J5008.2 (Pin_2), U5002.27 (GPIO16)
- new net IO18_L: J5008.3 (Pin_3), U5002.29 (GPIO18)
- new net LED_L: D5001.2 (A), U5002.28 (GPIO17)
- new net MISO_L: J5007.2 (Pin_2), U5002.31 (GPIO20)
- new net MOSI_L: J5004.4 (MOSI), J5007.5 (Pin_5), U5002.35 (GPIO23)
- new net M_COL1_L: D5002.3 (K), D5003.3 (K), U5002.11 (GPIO8)
- new net M_COL2_L: D5005.3 (K), D5006.3 (K), U5002.12 (GPIO9)
- new net M_COL3_L: D5007.3 (K), D5008.3 (K), U5002.9 (GPIO7)
- new net M_COL4_L: D5009.1 (K), D5010.3 (K), U5002.8 (GPIO6)
- new net M_COL5_L: D5011.1 (K), D5012.3 (K), U5002.40 (GPIO28_ADC2)
- new net M_ROW1_L: SW5005.1, SW5009.1, SW5013.1, SW5020.S2, U5002.38 (GPIO26_ADC0)
- new net M_ROW2_L: SW5002.1, SW5006.1, SW5010.1, SW5014.1, SW5017.1, U5002.6 (GPIO4)
- new net M_ROW3_L: SW5003.1, SW5007.1, SW5011.1, SW5015.1, SW5018.1, U5002.7 (GPIO5)
- new net M_ROW4_L: SW5004.1, SW5008.1, SW5012.1, SW5016.1, SW5019.1, U5002.39 (GPIO27_ADC1)
- new net NCS_L: J5007.3 (Pin_3), U5002.32 (GPIO21)
- new net QP_CS_L: J5004.6 (~{CS}), U5002.15 (GPIO12)
- new net QP_DC_L: J5004.5 (D/C), U5002.14 (GPIO11)
- new net QP_RST_L: J5004.7 (RST), U5002.16 (GPIO13)
- new net QSPI_D0_L: U5002.53 (QSPI_SD0), U5004.5 (DI(IO0))
- new net QSPI_D1_L: U5002.55 (QSPI_SD1), U5004.2 (DO(IO1))
- new net QSPI_D2_L: U5002.54 (QSPI_SD2), U5004.3 (IO2)
- new net QSPI_D3_L: U5002.51 (QSPI_SD3), U5004.7 (IO3)
- new net QSPI_SCLK_L: U5002.52 (QSPI_SCLK), U5004.6 (CLK)
- new net QSPI_~{CS}_L: R5003.2, R5011.1, U5002.56 (QSPI_SS), U5004.1 (~{CS})
- new net RGB_L: J5006.3 (Pin_3), U5002.2 (GPIO0)
- new net SCLK_L: J5004.3 (SCK), J5007.1 (Pin_1), U5002.34 (GPIO22)
- new net SCL_L: J5007.9 (Pin_9), O5001.3 (Pin_3), R5014.2, U5002.5 (GPIO3)
- new net SDA_L: J5007.10 (Pin_10), O5001.4 (Pin_4), R5013.1, U5002.4 (GPIO2)
- new net SERIAL_L: J5003.R2, U5002.3 (GPIO1)
- new net SWCLK_L: J5005.3 (Pin_3), U5002.24 (SWCLK)
- new net SWD_L: J5005.2 (Pin_2), U5002.25 (SWD)
- new net UNDER_RGB_L: D5013.1 (DIN), U5002.13 (GPIO10)
- new net VBUS_DET_L: R5009.1, R5010.2, U5002.30 (GPIO19)
- new net VBUS_L: F5001.1, J5001.A4 (VBUS), J5001.A9 (VBUS), J5001.B4 (VBUS), J5001.B9 (VBUS), R5009.2, U5003.5 (VBUS)
- new net encoder_diode_L: D5008.1 (A), SW5013.2, SW5020.S1
- new net ~{RESET_L}: J5008.4 (Pin_4), R5002.1, SW5001.2, U5002.26 (RUN/~{RST})
- no-connect marks 12 -> 24

Commit message: routing
Connections:
- net +3V3_L: no longer J5003.T
- net GND_L: now also J5003.T
Changed lines of the file:
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@@
     (effects (font (size 1.778 1.778) (thickness 0.3556) bold) (justify left bottom))
   )
-  (text "reverse for left half" (at 286.385 487.045 0)
-    (effects (font (size 1.27 1.27)) (justify left bottom))
-  )
   (text "Tenting puck" (at 365.76 166.37 180)
     (effects (font (size 1.778 1.778) (thickness 0.3556) bold) (justify right bottom))
@@
     (pin "2")
   )
-  (symbol (lib_id "power_L:+3V3_L") (at 289.56 475.615 0) (unit 1)
-    (in_bom yes) (on_board yes) (fields_autoplaced)
-    (property "Reference" "#PWR05047" (id 0) (at 289.56 479.425 0)
-      (effects (font (size 1.27 1.27)) hide)
-    )
-    (property "Value" "+3V3_L" (id 1) (at 289.56 470.535 0))
-    (property "Footprint" "" (id 2) (at 289.56 475.615 0)
-      (effects (font (size 1.27 1.27)) hide)
-    )
-    (property "Datasheet" "" (id 3) (at 289.56 475.615 0)
-      (effects (font (size 1.27 1.27)) hide)
-    )
-    (pin "1")
-  )
   (symbol (lib_id "Switch:SW_Push") (at 76.2 218.44 0) (unit 1)
     (in_bom yes) (on_board yes)
@@
     (pin "2")
   )
+  (symbol (lib_id "power_L:GND_L") (at 289.56 475.615 180) (unit 1)
+    (in_bom yes) (on_board yes) (fields_autoplaced)
+    (property "Reference" "#PWR?" (id 0) (at 289.56 469.265 0)
+      (effects (font (size 1.27 1.27)) hide)
+    )
+    (property "Value" "GND_L" (id 1) (at 291.465 474.3449 0)
+      (effects (font (size 1.27 1.27)) (justify right))
+    )
+    (property "Footprint" "" (id 2) (at 289.56 475.615 0)
+      (effects (font (size 1.27 1.27)) hide)
+    )
+    (property "Datasheet" "" (id 3) (at 289.56 475.615 0)
+      (effects (font (size 1.27 1.27)) hide)
+    )
+    (pin "1")
+  )
   (symbol (lib_id "power:GND") (at 226.695 179.07 0) (unit 1)
     (in_bom yes) (on_board yes)
@@
       (reference "#PWR05046") (unit 1) (value "+3V3_L") (footprint "")
     )
-    (path "/395f8c20-37fa-40d8-aee1-c7ff83eb9b73"
-      (reference "#PWR05047") (unit 1) (value "+3V3_L") (footprint "")
-    )
     (path "/13bc5665-b353-441d-9f36-59e1512015c5"
       (reference "#PWR05048") (unit 1) (value "GND_L") (footprint "")
@@
       (reference "#PWR05059") (unit 1) (value "GND_L") (footprint "")
     )
+    (path "/7dddb86e-fee6-4480-8dee-61b21e51504b"
+      (reference "#PWR?") (unit 1) (value "GND_L") (footprint "")
+    )
     (path "/4a21e78b-0ab0-4b88-8132-9b174e045719"

Commit message: routing
Connections:
- net +3V3_L: now also J5003.T; no longer R5012.2
- net GND_L: now also R5012.2; no longer J5003.T
Changed lines of the file:
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@@
     (stroke (width 0) (type default) (color 0 0 0 0))
   )
-  (wire (pts (xy 288.925 517.525) (xy 288.925 514.985))
-    (stroke (width 0) (type default) (color 0 0 0 0))
-  )
   (polyline (pts (xy 77.47 194.31) (xy 172.72 194.31))
     (stroke (width 0) (type default) (color 0 0 0 0))
@@
     (pin "2")
   )
+  (symbol (lib_id "power_L:GND_L") (at 288.925 517.525 0) (unit 1)
+    (in_bom yes) (on_board yes)
+    (property "Reference" "#PWR?" (id 0) (at 288.925 523.875 0)
+      (effects (font (size 1.27 1.27)) hide)
+    )
+    (property "Value" "GND_L" (id 1) (at 288.9249 516.89 0)
+      (effects (font (size 1.27 1.27)) (justify left))
+    )
+    (property "Footprint" "" (id 2) (at 288.925 517.525 0)
+      (effects (font (size 1.27 1.27)) hide)
+    )
+    (property "Datasheet" "" (id 3) (at 288.925 517.525 0)
+      (effects (font (size 1.27 1.27)) hide)
+    )
+    (pin "1")
+  )
   (symbol (lib_id "sk6805-ec15:SK6805-EC15") (at 526.415 351.155 0) (unit 1)
     (in_bom yes) (on_board yes)
@@
     (pin "4")
   )
+  (symbol (lib_id "power_L:+3V3_L") (at 289.56 475.615 0) (unit 1)
+    (in_bom yes) (on_board yes) (fields_autoplaced)
+    (property "Reference" "#PWR?" (id 0) (at 289.56 479.425 0)
+      (effects (font (size 1.27 1.27)) hide)
+    )
+    (property "Value" "+3V3_L" (id 1) (at 289.56 470.535 0))
+    (property "Footprint" "" (id 2) (at 289.56 475.615 0)
+      (effects (font (size 1.27 1.27)) hide)
+    )
+    (property "Datasheet" "" (id 3) (at 289.56 475.615 0)
+      (effects (font (size 1.27 1.27)) hide)
+    )
+    (pin "1")
+  )
   (symbol (lib_id "Device:C") (at 121.92 180.34 0) (unit 1)
     (in_bom yes) (on_board yes)
@@
     (pin "2")
   )
-  (symbol (lib_id "power_L:GND_L") (at 289.56 475.615 180) (unit 1)
-    (in_bom yes) (on_board yes) (fields_autoplaced)
-    (property "Reference" "#PWR?" (id 0) (at 289.56 469.265 0)
-      (effects (font (size 1.27 1.27)) hide)
-    )
-    (property "Value" "GND_L" (id 1) (at 291.465 474.3449 0)
-      (effects (font (size 1.27 1.27)) (justify right))
-    )
-    (property "Footprint" "" (id 2) (at 289.56 475.615 0)
-      (effects (font (size 1.27 1.27)) hide)
-    )
-    (property "Datasheet" "" (id 3) (at 289.56 475.615 0)
-      (effects (font (size 1.27 1.27)) hide)
-    )
-    (pin "1")
-  )
   (symbol (lib_id "power:GND") (at 226.695 179.07 0) (unit 1)
     (in_bom yes) (on_board yes)
@@
     (pin "2")
   )
-  (symbol (lib_id "power_L:+3V3_L") (at 288.925 514.985 0) (unit 1)
-    (in_bom yes) (on_board yes) (fields_autoplaced)
-    (property "Reference" "#PWR05046" (id 0) (at 288.925 518.795 0)
-      (effects (font (size 1.27 1.27)) hide)
-    )
-    (property "Value" "+3V3_L" (id 1) (at 288.925 509.905 0))
-    (property "Footprint" "" (id 2) (at 288.925 514.985 0)
-      (effects (font (size 1.27 1.27)) hide)
-    )
-    (property "Datasheet" "" (id 3) (at 288.925 514.985 0)
-      (effects (font (size 1.27 1.27)) hide)
-    )
-    (pin "1")
-  )
   (symbol (lib_id "Device:R") (at 37.465 462.915 180) (unit 1)
     (in_bom yes) (on_board yes)
@@
       (reference "#PWR05045") (unit 1) (value "GND_L") (footprint "")
     )
-    (path "/c081bcf0-3d52-428a-9f65-fc0388f04ed2"
-      (reference "#PWR05046") (unit 1) (value "+3V3_L") (footprint "")
-    )
     (path "/13bc5665-b353-441d-9f36-59e1512015c5"
       (reference "#PWR05048") (unit 1) (value "GND_L") (footprint "")
@@
       (reference "#PWR05059") (unit 1) (value "GND_L") (footprint "")
     )
-    (path "/7dddb86e-fee6-4480-8dee-61b21e51504b"
+    (path "/209147cd-5107-4e05-a842-782aab18be28"
       (reference "#PWR?") (unit 1) (value "GND_L") (footprint "")
     )
+    (path "/387a6227-b331-470e-ab79-9947b9ac881d"
+      (reference "#PWR?") (unit 1) (value "+3V3_L") (footprint "")
+    )
     (path "/4a21e78b-0ab0-4b88-8132-9b174e045719"
       (reference "C1") (unit 1) (value "1µ") (footprint "Capacitor_SMD:C_0603_1608Metric")
@@
       (reference "D5028") (unit 1) (value "SK6805-EC15") (footprint "0xB2_drawings:LED_SK6805-EC15_1.5x1.5mm_P0.6mm_handsolder(1)")
     )
-    (path "/20cb7a59-5c46-47a2-8fc8-a951f476d54d"
+    (path "/20cb7a59-5c46-47a2-8fc8-a951f476d54e"
       (reference "D5029") (unit 1) (value "SK6805-EC15") (footprint "0xB2_drawings:LED_SK6805-EC15_1.5x1.5mm_P0.6mm_handsolder(1)")
     )

Commit message: routing
Connections:
- net RGB: now also D5.3 (DOUT); no longer U1.2 (GPIO0)
- net RGB_L: now also D5015.3 (DOUT); no longer U5002.2 (GPIO0)
- net IO14_L: now reaches U5002.17 (GPIO14)
- net IO14_L: now also J5008.2 (Pin_2)
- net IO15_L: now reaches U5002.18 (GPIO15)
- net IO15_L: now also J5008.3 (Pin_3)
- net IO16_L: no longer names the net of U5002.27 (GPIO16)
- net IO16_L: no longer J5008.2 (Pin_2)
- net IO18_L: no longer names the net of U5002.29 (GPIO18)
- net IO18_L: no longer J5008.3 (Pin_3)
Changed lines of the file:
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@@
   (junction (at 399.415 321.945) (diameter 0) (color 0 0 0 0)
   )
+  (no_connect (at 180.34 394.335))
   (no_connect (at 342.265 50.8))
   (no_connect (at 342.265 40.64))
@@
   (no_connect (at 342.265 60.96))
   (no_connect (at 342.265 63.5))
-  (no_connect (at 180.34 389.255))
+  (no_connect (at 180.34 353.695))
   (no_connect (at 339.725 340.995))
   (no_connect (at 265.43 176.53))
@@
   (no_connect (at 182.88 93.98))
   (no_connect (at 182.88 96.52))
-  (no_connect (at 409.575 74.93))
+  (no_connect (at 182.88 58.42))
   (no_connect (at 339.725 346.075))
   (no_connect (at 339.725 335.915))
   (no_connect (at 48.26 360.045))
-  (no_connect (at 407.035 370.205))
+  (no_connect (at 180.34 399.415))
   (no_connect (at 339.725 338.455))
-  (no_connect (at 180.34 391.795))
   (no_connect (at 339.725 356.235))
   (no_connect (at 339.725 358.775))
@@
     )
   )
-  (global_label "RGB_L" (shape input) (at 180.34 353.695 0)
-    (effects (font (size 1.27 1.27)) (justify left))
-    (property "Intersheet References" "${INTERSHEET_REFS}" (id 0) (at 267.97 421.005 0)
-      (effects (font (size 1.27 1.27)) hide)
-    )
-  )
   (global_label "M_COL3" (shape input) (at 182.88 76.2 0)
     (effects (font (size 1.27 1.27)) (justify left))
@@
     )
   )
-  (global_label "IO16_L" (shape input) (at 434.34 407.67 180) (fields_autoplaced)
+  (global_label "IO14_L" (shape input) (at 434.34 407.67 180) (fields_autoplaced)
     (effects (font (size 1.27 1.27)) (justify right))
-    (property "Intersheet References" "${INTERSHEET_REFS}" (id 0) (at 427.5726 407.7494 0)
+    (property "Intersheet References" "${INTERSHEET_REFS}" (id 0) (at 425.5769 407.5906 0)
       (effects (font (size 1.27 1.27)) (justify right) hide)
     )
@@
     )
   )
-  (global_label "IO18_L" (shape input) (at 434.34 410.21 180) (fields_autoplaced)
+  (global_label "IO15_L" (shape input) (at 434.34 410.21 180) (fields_autoplaced)
     (effects (font (size 1.27 1.27)) (justify right))
-    (property "Intersheet References" "${INTERSHEET_REFS}" (id 0) (at 427.5726 410.2894 0)
+    (property "Intersheet References" "${INTERSHEET_REFS}" (id 0) (at 425.5769 410.1306 0)
       (effects (font (size 1.27 1.27)) (justify right) hide)
     )
   )
+  (global_label "RGB_L" (shape input) (at 407.035 370.205 0)
+    (effects (font (size 1.27 1.27)) (justify left))
+    (property "Intersheet References" "${INTERSHEET_REFS}" (id 0) (at 494.665 437.515 0)
+      (effects (font (size 1.27 1.27)) hide)
+    )
+  )
   (global_label "SDA" (shape input) (at 329.565 35.56 180)
     (effects (font (size 1.27 1.27)) (justify right))
@@
     )
   )
-  (global_label "IO18_L" (shape input) (at 180.34 399.415 0) (fields_autoplaced)
+  (global_label "IO15_L" (shape input) (at 180.34 391.795 0) (fields_autoplaced)
     (effects (font (size 1.27 1.27)) (justify left))
-    (property "Intersheet References" "${INTERSHEET_REFS}" (id 0) (at 187.1074 399.3356 0)
+    (property "Intersheet References" "${INTERSHEET_REFS}" (id 0) (at 189.1031 391.7156 0)
       (effects (font (size 1.27 1.27)) (justify left) hide)
     )
@@
     )
   )
-  (global_label "RGB" (shape input) (at 182.88 58.42 0)
-    (effects (font (size 1.27 1.27)) (justify left))
-    (property "Intersheet References" "${INTERSHEET_REFS}" (id 0) (at 270.51 125.73 0)
-      (effects (font (size 1.27 1.27)) hide)
-    )
-  )
   (global_label "M_COL2_L" (shape input) (at 180.34 376.555 0)
     (effects (font (size 1.27 1.27)) (justify left))
@@
     )
   )
-  (global_label "IO16_L" (shape input) (at 180.34 394.335 0) (fields_autoplaced)
+  (global_label "IO14_L" (shape input) (at 180.34 389.255 0) (fields_autoplaced)
     (effects (font (size 1.27 1.27)) (justify left))
-    (property "Intersheet References" "${INTERSHEET_REFS}" (id 0) (at 187.1074 394.2556 0)
+    (property "Intersheet References" "${INTERSHEET_REFS}" (id 0) (at 189.1031 389.1756 0)
       (effects (font (size 1.27 1.27)) (justify left) hide)
     )
@@
     )
   )
+  (global_label "RGB" (shape input) (at 409.575 74.93 0)
+    (effects (font (size 1.27 1.27)) (justify left))
+    (property "Intersheet References" "${INTERSHEET_REFS}" (id 0) (at 497.205 142.24 0)
+      (effects (font (size 1.27 1.27)) hide)
+    )
+  )
   (global_label "SERIAL" (shape input) (at 182.88 60.96 0)
     (effects (font (size 1.27 1.27)) (justify left))
@@
   (symbol (lib_id "power_L:GND_L") (at 288.925 517.525 0) (unit 1)
     (in_bom yes) (on_board yes)
-    (property "Reference" "#PWR?" (id 0) (at 288.925 523.875 0)
+    (property "Reference" "#PWR0116" (id 0) (at 288.925 523.875 0)
       (effects (font (size 1.27 1.27)) hide)
     )
@@
   (symbol (lib_id "power_L:+3V3_L") (at 289.56 475.615 0) (unit 1)
     (in_bom yes) (on_board yes) (fields_autoplaced)
-    (property "Reference" "#PWR?" (id 0) (at 289.56 479.425 0)
+    (property "Reference" "#PWR0119" (id 0) (at 289.56 479.425 0)
       (effects (font (size 1.27 1.27)) hide)
     )
@@
       (reference "#PWR0115") (unit 1) (value "+3.3V") (footprint "")
     )
+    (path "/209147cd-5107-4e05-a842-782aab18be28"
+      (reference "#PWR0116") (unit 1) (value "GND_L") (footprint "")
+    )
     (path "/65cc9c59-39dc-4148-a69b-a97364bae0ce"
       (reference "#PWR0117") (unit 1) (value "+3.3V") (footprint "")
@@
       (reference "#PWR0118") (unit 1) (value "+3.3V") (footprint "")
     )
+    (path "/387a6227-b331-470e-ab79-9947b9ac881d"
+      (reference "#PWR0119") (unit 1) (value "+3V3_L") (footprint "")
+    )
     (path "/6564800d-9dea-4777-82f3-5251944a6f28"
       (reference "#PWR0120") (unit 1) (value "+3.3V") (footprint "")
@@
       (reference "#PWR05059") (unit 1) (value "GND_L") (footprint "")
     )
-    (path "/209147cd-5107-4e05-a842-782aab18be28"
-      (reference "#PWR?") (unit 1) (value "GND_L") (footprint "")
-    )
-    (path "/387a6227-b331-470e-ab79-9947b9ac881d"
-      (reference "#PWR?") (unit 1) (value "+3V3_L") (footprint "")
-    )
     (path "/4a21e78b-0ab0-4b88-8132-9b174e045719"

Commit message: connect rgb R
Parts:
- added C5015, C5016, C5017, C?: 1µ, Capacitor_SMD:C_0402_1005Metric, symbol Device:C
- added D5031, D5032, D5033, D5034, D5035, D5036, D5037, D5038, D5039, D5040, D5041, D5042, D5043, D5044, D5045, D5046, D5047, D5048, D? (x18): SK6812MINI, local-libraries:SK6812_mini_e_corners, symbol LED:SK6812MINI
- added J5009, J5010: Conn_01x05, local-libraries:PinHeader_1x05_P1.27mm_Vertical_SMD, symbol Connector_Generic:Conn_01x05
- added R5015, R5016: 1k, Resistor_SMD:R_0402_1005Metric, symbol Device:R
- added SW5021, SW5022: SW_SPST, Library:PushSwitch, symbol Switch:SW_SPST
Connections:
- net +3V3: now also C5015.1, C5017.1, D5031.4 (VDD), D5032.4 (VDD), D5033.4 (VDD), D5034.4 (VDD), D5035.4 (VDD), D5036.4 (VDD), D5037.4 (VDD), D5038.4 (VDD), D5039.4 (VDD), D5040.4 (VDD), D5041.4 (VDD), D5042.4 (VDD), D5043.4 (VDD), D5044.4 (VDD), D5045.4 (VDD), D5046.4 (VDD), D5047.4 (VDD), D5048.4 (VDD), J5010.1 (Pin_1); no longer D12.2 (VDD), D16.2 (VDD), D19.2 (VDD), D22.2 (VDD), D25.2 (VDD), D28.2 (VDD), D4.2 (VDD), D5.2 (VDD), D8.2 (VDD), D9.2 (VDD)
- net +3V3_L: now also C5016.1, C?.1, D?.4 (VDD), D?.4 (VDD), D?.4 (VDD), D?.4 (VDD), D?.4 (VDD), D?.4 (VDD), D?.4 (VDD), D?.4 (VDD), D?.4 (VDD), D?.4 (VDD), D?.4 (VDD), D?.4 (VDD), D?.4 (VDD), D?.4 (VDD), D?.4 (VDD), D?.4 (VDD), D?.4 (VDD), D?.4 (VDD), J5009.1 (Pin_1); no longer D5014.2 (VDD), D5015.2 (VDD), D5017.2 (VDD), D5019.2 (VDD), D5021.2 (VDD), D5023.2 (VDD), D5025.2 (VDD), D5027.2 (VDD), D5029.2 (VDD), D5030.2 (VDD)
- net GND: now also C5015.2, C5017.2, D5031.2 (VSS), D5032.2 (VSS), D5033.2 (VSS), D5034.2 (VSS), D5035.2 (VSS), D5036.2 (VSS), D5037.2 (VSS), D5038.2 (VSS), D5039.2 (VSS), D5040.2 (VSS), D5041.2 (VSS), D5042.2 (VSS), D5043.2 (VSS), D5044.2 (VSS), D5045.2 (VSS), D5046.2 (VSS), D5047.2 (VSS), D5048.2 (VSS), J5010.5 (Pin_5), SW5022.2 (B)
- net GND_L: now also C5016.2, C?.2, D?.2 (VSS), D?.2 (VSS), D?.2 (VSS), D?.2 (VSS), D?.2 (VSS), D?.2 (VSS), D?.2 (VSS), D?.2 (VSS), D?.2 (VSS), D?.2 (VSS), D?.2 (VSS), D?.2 (VSS), D?.2 (VSS), D?.2 (VSS), D?.2 (VSS), D?.2 (VSS), D?.2 (VSS), D?.2 (VSS), J5009.5 (Pin_5), SW5021.2 (B)
- net IO14_L: now also J5009.2 (Pin_2)
- net IO15_L: now also J5009.3 (Pin_3)
- net IO16: now also J5010.2 (Pin_2)
- net IO18: now also J5010.3 (Pin_3)
- net RGB: now also D5031.3 (DIN)
- net RGB_L: now also D?.3 (DIN)
- net UNDER_RGB: now also R5016.1; no longer D3.1 (DIN)
- net UNDER_RGB_L: now also R5015.1; no longer D5013.1 (DIN)
- net ~{RESET_L}: now also J5009.4 (Pin_4), SW5021.1 (A)
- net ~{RESET}: now also J5010.4 (Pin_4), SW5022.1 (A)
- new net: D12.2 (VDD), D16.2 (VDD), D19.2 (VDD), D22.2 (VDD), D25.2 (VDD), D28.2 (VDD), D4.2 (VDD), D5.2 (VDD), D8.2 (VDD), D9.2 (VDD)
- new net: D?.1 (DOUT), D?.3 (DIN) (x17)
- new net: D5031.1 (DOUT), D5034.3 (DIN)
- new net: D5014.2 (VDD), D5015.2 (VDD), D5017.2 (VDD), D5019.2 (VDD), D5021.2 (VDD), D5023.2 (VDD), D5025.2 (VDD), D5027.2 (VDD), D5029.2 (VDD), D5030.2 (VDD)
- new net: D5033.3 (DIN), D5048.1 (DOUT)
- new net: D5036.1 (DOUT), D5038.3 (DIN)
- new net: D5034.1 (DOUT), D5036.3 (DIN)
- new net: D5040.1 (DOUT), D5042.3 (DIN)
- new net: D5038.1 (DOUT), D5040.3 (DIN)
- new net: D5047.1 (DOUT), D5048.3 (DIN)
- new net: D5032.1 (DOUT), D5035.3 (DIN)
- new net: D5032.3 (DIN), D5046.1 (DOUT)
- new net: D5013.1 (DIN), R5015.2
- new net: D5043.1 (DOUT), D5045.3 (DIN)
- new net: D5041.1 (DOUT), D5043.3 (DIN)
- new net: D5035.1 (DOUT), D5037.3 (DIN)
- new net: D3.1 (DIN), R5016.2
- new net: D5039.1 (DOUT), D5041.3 (DIN)
- new net: D5037.1 (DOUT), D5039.3 (DIN)
- new net: D5045.1 (DOUT), D5047.3 (DIN)
- new net: D5044.1 (DOUT), D5046.3 (DIN)
- new net: D5042.1 (DOUT), D5044.3 (DIN)
- no-connect marks 24 -> 26
Other:
- note added: "Per key RGB"
- note added: "RST button"
- moved on the sheet: D11, D12, D15, D16, D18, D19, D21, D22, D24, D25, D27, D28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
